Commit message: Fixed z value for initial pose of robotic arm in house.world

File: mycobot_gazebo/urdf/mycobot_280_classic_gazebo.urdf.xacro (robot description, xacro)
@@ -413,4 +413,5 @@
 		<child link="link2"/>
 		<origin xyz= "0 0 0.13156" rpy = "0 0 ${pi/2}"/>
+        <dynamics damping="8.0" friction="4.0"/>
 	</joint>
 	<joint name="link2_to_link3" type="revolute">
@@ -420,4 +421,5 @@
 		<child link="link3"/>
 		<origin xyz= "0 0 -0.001" rpy = "0 ${pi/2} ${-pi/2}"/>
+        <dynamics damping="8.0" friction="4.0"/>
 	</joint>
 	<joint name="link3_to_link4" type="revolute">
@@ -427,4 +429,5 @@
 		<child link="link4"/>
 		<origin xyz= "-0.1104 0 0   " rpy = "0 0 0"/>
+        <dynamics damping="8.0" friction="4.0"/>
 	</joint>
 	<joint name="link4_to_link5" type="revolute">
@@ -434,4 +437,5 @@
 		<child link="link5"/>
 		<origin xyz= "-0.096 0 0.06062" rpy = "0 0 ${-pi/2}"/>
+        <dynamics damping="8.0" friction="4.0"/>
 	</joint>
 	<joint name="link5_to_link6" type="revolute">
@@ -441,4 +445,5 @@
 		<child link="link6"/>
 		<origin xyz= "0 -0.07318 0" rpy = "${pi/2} ${-pi/2} 0"/>
+        <dynamics damping="5.0" friction="2.5"/>
 	</joint>
 	<joint name="link6_to_link6flange" type="revolute">
@@ -448,4 +453,5 @@
 		<child link="link6_flange"/>
 		<origin xyz= "0 0.0456 0" rpy = "${-pi/2} 0 0"/>
+        <dynamics damping="2.0" friction="1.5"/>
 	</joint>
 	<joint name="link6flange_to_gripper_base" type="fixed">
@@ -460,4 +466,5 @@
 		<child link="gripper_left3"/>
 		<origin xyz= "-0.012 0.005 0" rpy = "0 0 0"/>
+        <dynamics damping="3.0" friction="6.0"/>
 	</joint>
 	<!-- The mimic element means this joint will follow the movements of the
@@ -471,4 +478,5 @@
 		<origin xyz= "-0.005 0.027 0" rpy = "0 0 0"/>
 		<mimic joint="gripper_controller" multiplier="1.0" offset="0" />
+        <dynamics damping="3.0" friction="6.0"/>
 	</joint>
 	<joint name="gripper_left3_to_gripper_left1" type="revolute">
@@ -479,4 +487,5 @@
 		<origin xyz= "-0.027 0.016 0" rpy = "0 0 0"/>
 		<mimic joint="gripper_controller" multiplier="-1.0" offset="0" />
+        <dynamics damping="3.0" friction="6.0"/>
 	</joint>
 	<joint name="gripper_base_to_gripper_right3" type="revolute">
@@ -487,4 +496,5 @@
 		<origin xyz= "0.012 0.005 0" rpy = "0 0 0"/>
 		<mimic joint="gripper_controller" multiplier="-1.0" offset="0" />
+        <dynamics damping="3.0" friction="6.0"/>
 	</joint>
 	<joint name="gripper_base_to_gripper_right2" type="revolute">
@@ -495,4 +505,5 @@
 		<origin xyz= "0.005 0.027 0" rpy = "0 0 0"/>
 		<mimic joint="gripper_controller" multiplier="-1.0" offset="0" />
+        <dynamics damping="3.0" friction="6.0"/>
 	</joint>
 	<joint name="gripper_right3_to_gripper_right1" type="revolute">
@@ -503,4 +514,5 @@
 		<origin xyz= "0.027 0.016 0" rpy = "0 0 0"/>
 		<mimic joint="gripper_controller" multiplier="1.0" offset="0" />
+        <dynamics damping="3.0" friction="6.0"/>
 	</joint>
     <!-- Publishes joint state information for the model which the robot_state_publisher uses to broadcast to

Commit message: Added damping and friction to the robotic arms

File: mycobot_gazebo/urdf/mycobot_280_classic_gazebo.urdf.xacro (robot description, xacro)
@@ -24,8 +24,8 @@
 	<xacro:property name="velocity" value="2.792527"/>
 	<!-- ********** LINKS ********** -->
-    <!-- Define the base plate of the robotic arm -->
+    <!-- Define the base plate of the robotic arm
+    	The inertial values below were taken from link1 (with slight modification.
+		They are just placeholder values. -->
 	<link name="base_link">
-		<!-- The inertial values below were taken from link1 (with slight modification.
-		They are just placeholder values. -->
 		<inertial>
 			<origin xyz="0 0 0.0" rpy="0 0 0"/>
@@ -51,15 +51,7 @@
 	<!--Define the first link of the robotic arm. Each link represents a solid part of the robot.-->
 	<link name="link1">
-		<!--Define the inertial properties of the link, which characterizes the link's resistance
-		to changes in its rotational motion.-->
-		<inertial>
-			<!--Specify the pose of the center of mass of the link relative
-			to this link's coordinate frame.-->
-			<origin xyz="0 0 0.0" rpy="0 0 0"/>
-			<!--The mass of the link in kilograms-->
+		<inertial>
+			<origin xyz="0 0 0.0" rpy="0 0 0"/>
 			<mass value="0.12"/>
-			<!--The rotational inertia values, which reflect how easily the link can rotate around
-			different axes given the distribution of mass within the link. Here we see rotation is
-			most difficult around the y axis.-->
 			<inertia
 				ixx="0.000148" ixy="0.0" ixz="0.0"
@@ -67,18 +59,10 @@
 				izz="0.000096"/>
 		</inertial>
-		<!--Define the visual representation of the link in simulation.-->
-		<visual>
-			<!--Define the shape of the link-->
-			<geometry>
-				<!--Specify the link's visual appearance using the 3D mesh file.-->
+		<visual>
+			<geometry>
 				<mesh filename="file://$(find mycobot_description)/meshes/mycobot_280/link1.dae"/>
 			</geometry>
-			<!--Define the position and orientation of the visual representation relative to the
-			link's reference frame. Here, it's rotated by -1.5708 radians (or -90 degrees)
-			around the Z-axis.-->
 			<origin xyz = "0.0 0 0 " rpy = " 0 0 ${-pi/2}"/>
 		</visual>
-		<!--Define the shape used for collision detection during simulation. This piece is important
-		for accurate physical interactions between robot components and the environment or other objects.-->
 		<collision>
 			<geometry>
@@ -375,4 +359,32 @@
 		</collision>
 	</link>
+    <!-- ********** COLORS ********** -->
+    <gazebo reference="base_link">
+        <material>Gazebo/Grey</material>
+    </gazebo>
+    <gazebo reference="link1">
+        <material>Gazebo/White</material>
+    </gazebo>
+    <gazebo reference="link2">
+        <material>Gazebo/White</material>
+    </gazebo>
+    <gazebo reference="link3">
+        <material>Gazebo/White</material>
+    </gazebo>
+    <gazebo reference="link4">
+        <material>Gazebo/White</material>
+    </gazebo>
+    <gazebo reference="link5">
+        <material>Gazebo/White</material>
+    </gazebo>
+    <gazebo reference="link6">
+        <material>Gazebo/White</material>
+    </gazebo>
+    <gazebo reference="link6_flange">
+        <material>Gazebo/White</material>
+    </gazebo>
+    <gazebo reference="gripper_base">
+        <material>Gazebo/White</material>
+    </gazebo>
 	<!-- ********** JOINTS ********** -->
 	<!-- Attach the robot base to the world frame with no initial offset or rotation. -->
@@ -385,24 +397,8 @@
 	means the two connected links cannot move relative to each other. -->
 	<joint name="base_link_to_link1" type="fixed">
-		<!-- Specifies the axis around which the joint could rotate if it wasn't fixed. -->
 		<axis xyz="0 0 0"/>
-		<!-- Specifies the range of allowed motion if the joint wasn't fixed.
-			effort: Maximum torque in Nm
-			lower: Minimum allowed angle in radians
-			upper: Maximum allowed angle in radians
-			velocity: Maximum allowed angular velocity in radians per second (ignored for fixed joints)
-		-->
 		<limit effort = "${effort}" lower = "${-pi}" upper = "${pi}" velocity = "${velocity}"/>
-		<!-- The link this joint connects to on one side -->
 		<parent link="base_link"/>
-		<!-- The link this joint connects to on the other side -->
 		<child link="link1"/>
-		<!-- The origin of the joint relative to the parent link's coordinate frame.
-			xyz: The position of the child link relative to the parent link's coordinate frame.
-			rpy: The orientation of the child link relative to the parent link's coordinate frame.
-			See these posts for more information on coordinate frames in robotics:
-			https://automaticaddison.com/coordinate-frames-and-transforms-for-ros-based-mobile-robots/
-			https://automaticaddison.com/yaw-pitch-and-roll-diagrams-using-2d-coordinate-systems/
-		-->
 		<origin xyz= "0 0 0" rpy = "0 0 0"/>
 	</joint>
@@ -413,5 +409,5 @@
 		<child link="link2"/>
 		<origin xyz= "0 0 0.13156" rpy = "0 0 ${pi/2}"/>
-        <dynamics damping="8.0" friction="4.0"/>
+        <dynamics damping="12.0" friction="6.0"/>
 	</joint>
 	<joint name="link2_to_link3" type="revolute">
@@ -421,5 +417,5 @@
 		<child link="link3"/>
 		<origin xyz= "0 0 -0.001" rpy = "0 ${pi/2} ${-pi/2}"/>
-        <dynamics damping="8.0" friction="4.0"/>
+        <dynamics damping="12.0" friction="6.0"/>
 	</joint>
 	<joint name="link3_to_link4" type="revolute">
@@ -429,5 +425,5 @@
 		<child link="link4"/>
 		<origin xyz= "-0.1104 0 0   " rpy = "0 0 0"/>
-        <dynamics damping="8.0" friction="4.0"/>
+        <dynamics damping="12.0" friction="6.0"/>
 	</joint>
 	<joint name="link4_to_link5" type="revolute">
@@ -437,5 +433,5 @@
 		<child link="link5"/>
 		<origin xyz= "-0.096 0 0.06062" rpy = "0 0 ${-pi/2}"/>
-        <dynamics damping="8.0" friction="4.0"/>
+        <dynamics damping="12.0" friction="6.0"/>
 	</joint>
 	<joint name="link5_to_link6" type="revolute">
@@ -445,5 +441,5 @@
 		<child link="link6"/>
 		<origin xyz= "0 -0.07318 0" rpy = "${pi/2} ${-pi/2} 0"/>
-        <dynamics damping="5.0" friction="2.5"/>
+        <dynamics damping="7.0" friction="4.0"/>
 	</joint>
 	<joint name="link6_to_link6flange" type="revolute">
@@ -453,5 +449,5 @@
 		<child link="link6_flange"/>
 		<origin xyz= "0 0.0456 0" rpy = "${-pi/2} 0 0"/>
-        <dynamics damping="2.0" friction="1.5"/>
+        <dynamics damping="3.0" friction="3.0"/>
 	</joint>
 	<joint name="link6flange_to_gripper_base" type="fixed">
@@ -466,5 +462,5 @@
 		<child link="gripper_left3"/>
 		<origin xyz= "-0.012 0.005 0" rpy = "0 0 0"/>
-        <dynamics damping="3.0" friction="6.0"/>
+        <dynamics damping="2.0" friction="4.0"/>
 	</joint>
 	<!-- The mimic element means this joint will follow the movements of the
@@ -478,5 +474,5 @@
 		<origin xyz= "-0.005 0.027 0" rpy = "0 0 0"/>
 		<mimic joint="gripper_controller" multiplier="1.0" offset="0" />
-        <dynamics damping="3.0" friction="6.0"/>
+        <dynamics damping="2.0" friction="4.0"/>
 	</joint>
 	<joint name="gripper_left3_to_gripper_left1" type="revolute">
@@ -487,5 +483,5 @@
 		<origin xyz= "-0.027 0.016 0" rpy = "0 0 0"/>
 		<mimic joint="gripper_controller" multiplier="-1.0" offset="0" />
-        <dynamics damping="3.0" friction="6.0"/>
+        <dynamics damping="2.0" friction="4.0"/>
 	</joint>
 	<joint name="gripper_base_to_gripper_right3" type="revolute">
@@ -496,5 +492,5 @@
 		<origin xyz= "0.012 0.005 0" rpy = "0 0 0"/>
 		<mimic joint="gripper_controller" multiplier="-1.0" offset="0" />
-        <dynamics damping="3.0" friction="6.0"/>
+        <dynamics damping="2.0" friction="4.0"/>
 	</joint>
 	<joint name="gripper_base_to_gripper_right2" type="revolute">
@@ -505,5 +501,5 @@
 		<origin xyz= "0.005 0.027 0" rpy = "0 0 0"/>
 		<mimic joint="gripper_controller" multiplier="-1.0" offset="0" />
-        <dynamics damping="3.0" friction="6.0"/>
+        <dynamics damping="2.0" friction="4.0"/>
 	</joint>
 	<joint name="gripper_right3_to_gripper_right1" type="revolute">
@@ -514,5 +510,5 @@
 		<origin xyz= "0.027 0.016 0" rpy = "0 0 0"/>
 		<mimic joint="gripper_controller" multiplier="1.0" offset="0" />
-        <dynamics damping="3.0" friction="6.0"/>
+        <dynamics damping="2.0" friction="4.0"/>
 	</joint>
     <!-- Publishes joint state information for the model which the robot_state_publisher uses to broadcast to

File: mycobot_gazebo/urdf/mycobot_280_gazebo.urdf.xacro (robot description, xacro)
@@ -412,5 +412,6 @@
 		<parent link="link1"/>
 		<child link="link2"/>
-		<origin xyz= "0 0 0.13156" rpy = "0 0 ${pi/2}"/>
+	    <origin xyz= "0 0 0.13156" rpy = "0 0 ${pi/2}"/>
+        <dynamics damping="12.0" friction="6.0"/>
 	</joint>
 	<joint name="link2_to_link3" type="revolute">
@@ -420,4 +421,5 @@
 		<child link="link3"/>
 		<origin xyz= "0 0 -0.001" rpy = "0 ${pi/2} ${-pi/2}"/>
+        <dynamics damping="12.0" friction="6.0"/>
 	</joint>
 	<joint name="link3_to_link4" type="revolute">
@@ -427,4 +429,5 @@
 		<child link="link4"/>
 		<origin xyz= "-0.1104 0 0   " rpy = "0 0 0"/>
+        <dynamics damping="12.0" friction="6.0"/>
 	</joint>
 	<joint name="link4_to_link5" type="revolute">
@@ -434,4 +437,5 @@
 		<child link="link5"/>
 		<origin xyz= "-0.096 0 0.06062" rpy = "0 0 ${-pi/2}"/>
+        <dynamics damping="12.0" friction="6.0"/>
 	</joint>
 	<joint name="link5_to_link6" type="revolute">
@@ -441,4 +445,5 @@
 		<child link="link6"/>
 		<origin xyz= "0 -0.07318 0" rpy = "${pi/2} ${-pi/2} 0"/>
+        <dynamics damping="7.0" friction="4.0"/>
 	</joint>
 	<joint name="link6_to_link6flange" type="revolute">
@@ -448,4 +453,5 @@
 		<child link="link6_flange"/>
 		<origin xyz= "0 0.0456 0" rpy = "${-pi/2} 0 0"/>
+        <dynamics damping="3.0" friction="3.0"/>
 	</joint>
 	<joint name="link6flange_to_gripper_base" type="fixed">
@@ -460,4 +466,5 @@
 		<child link="gripper_left3"/>
 		<origin xyz= "-0.012 0.005 0" rpy = "0 0 0"/>
+        <dynamics damping="2.0" friction="4.0"/>
 	</joint>
 	<!-- The mimic element means this joint will follow the movements of the
@@ -471,4 +478,5 @@
 		<origin xyz= "-0.005 0.027 0" rpy = "0 0 0"/>
 		<mimic joint="gripper_controller" multiplier="1.0" offset="0" />
+        <dynamics damping="2.0" friction="4.0"/>
 	</joint>
 	<joint name="gripper_left3_to_gripper_left1" type="revolute">
@@ -479,4 +487,5 @@
 		<origin xyz= "-0.027 0.016 0" rpy = "0 0 0"/>
 		<mimic joint="gripper_controller" multiplier="-1.0" offset="0" />
+        <dynamics damping="2.0" friction="4.0"/>
 	</joint>
 	<joint name="gripper_base_to_gripper_right3" type="revolute">
@@ -487,4 +496,5 @@
 		<origin xyz= "0.012 0.005 0" rpy = "0 0 0"/>
 		<mimic joint="gripper_controller" multiplier="-1.0" offset="0" />
+        <dynamics damping="2.0" friction="4.0"/>
 	</joint>
 	<joint name="gripper_base_to_gripper_right2" type="revolute">
@@ -495,4 +505,5 @@
 		<origin xyz= "0.005 0.027 0" rpy = "0 0 0"/>
 		<mimic joint="gripper_controller" multiplier="-1.0" offset="0" />
+        <dynamics damping="2.0" friction="4.0"/>
 	</joint>
 	<joint name="gripper_right3_to_gripper_right1" type="revolute">
@@ -503,4 +514,5 @@
 		<origin xyz= "0.027 0.016 0" rpy = "0 0 0"/>
 		<mimic joint="gripper_controller" multiplier="1.0" offset="0" />
+        <dynamics damping="2.0" friction="4.0"/>
 	</joint>
     <!-- JointStatePublisher publishes joint state information for the model -->
