Commit message: Created joint position publisher for new Gazebo implementation

File: mycobot_gazebo/urdf/mycobot_280_classic_gazebo.urdf.xacro (robot description, xacro)
@@ -512,4 +512,5 @@
         <dynamics damping="2.0" friction="4.0"/>
 	</joint>
+	<!-- ********** PLUGINS ********** -->
     <!-- Publishes joint state information for the model which the robot_state_publisher uses to broadcast to
             the tf topic, the topic that keeps track of the robot's multiple coordinate frames over time -->
@@ -524,5 +525,19 @@
             <joint_name>link6_to_link6flange</joint_name>
             <joint_name>gripper_controller</joint_name>
+            <joint_name>gripper_base_to_gripper_left2</joint_name>
+            <joint_name>gripper_left3_to_gripper_left1</joint_name>
+            <joint_name>gripper_base_to_gripper_right3</joint_name>
+            <joint_name>gripper_base_to_gripper_right2</joint_name>
+            <joint_name>gripper_right3_to_gripper_right1</joint_name>
         </plugin>
     </gazebo>
+    <!-- Subscribes to a JointTrajectory message from the /set_joint_trajectory topic
+        To publish to this topic type:
+            ros2 topic pub -1 /set_joint_trajectory trajectory_msgs/msg/JointTrajectory "{header: {frame_id: base_link}, joint_names: [link1_to_link2, link2_to_link3, etc.], points: [{positions: [0.0,0.0,etc.]}]}"
+    -->
+    <gazebo>
+        <plugin name="gazebo_ros_joint_pose_trajectory" filename="libgazebo_ros_joint_pose_trajectory.so">
+            <update_rate>20</update_rate>
+        </plugin>
+    </gazebo>
 </robot>

File: mycobot_gazebo/urdf/mycobot_280_gazebo.urdf.xacro (robot description, xacro)
@@ -413,5 +413,5 @@
 		<child link="link2"/>
 	    <origin xyz= "0 0 0.13156" rpy = "0 0 ${pi/2}"/>
-        <dynamics damping="12.0" friction="6.0"/>
+        <dynamics damping="0.05" friction="0.05"/>
 	</joint>
 	<joint name="link2_to_link3" type="revolute">
@@ -421,5 +421,5 @@
 		<child link="link3"/>
 		<origin xyz= "0 0 -0.001" rpy = "0 ${pi/2} ${-pi/2}"/>
-        <dynamics damping="12.0" friction="6.0"/>
+        <dynamics damping="0.205" friction="0.515"/>
 	</joint>
 	<joint name="link3_to_link4" type="revolute">
@@ -429,5 +429,5 @@
 		<child link="link4"/>
 		<origin xyz= "-0.1104 0 0   " rpy = "0 0 0"/>
-        <dynamics damping="12.0" friction="6.0"/>
+        <dynamics damping="0.21" friction="0.41"/>
 	</joint>
 	<joint name="link4_to_link5" type="revolute">
@@ -437,5 +437,5 @@
 		<child link="link5"/>
 		<origin xyz= "-0.096 0 0.06062" rpy = "0 0 ${-pi/2}"/>
-        <dynamics damping="12.0" friction="6.0"/>
+        <dynamics damping="0.10" friction="0.20"/>
 	</joint>
 	<joint name="link5_to_link6" type="revolute">
@@ -445,5 +445,5 @@
 		<child link="link6"/>
 		<origin xyz= "0 -0.07318 0" rpy = "${pi/2} ${-pi/2} 0"/>
-        <dynamics damping="7.0" friction="4.0"/>
+        <dynamics damping="0.01" friction="0.005"/>
 	</joint>
 	<joint name="link6_to_link6flange" type="revolute">
@@ -453,5 +453,5 @@
 		<child link="link6_flange"/>
 		<origin xyz= "0 0.0456 0" rpy = "${-pi/2} 0 0"/>
-        <dynamics damping="3.0" friction="3.0"/>
+        <dynamics damping="0.01" friction="0.005"/>
 	</joint>
 	<joint name="link6flange_to_gripper_base" type="fixed">
@@ -466,5 +466,5 @@
 		<child link="gripper_left3"/>
 		<origin xyz= "-0.012 0.005 0" rpy = "0 0 0"/>
-        <dynamics damping="2.0" friction="4.0"/>
+        <dynamics damping="0.01" friction="0.005"/>
 	</joint>
 	<!-- The mimic element means this joint will follow the movements of the
@@ -478,5 +478,5 @@
 		<origin xyz= "-0.005 0.027 0" rpy = "0 0 0"/>
 		<mimic joint="gripper_controller" multiplier="1.0" offset="0" />
-        <dynamics damping="2.0" friction="4.0"/>
+        <dynamics damping="0.01" friction="0.005"/>
 	</joint>
 	<joint name="gripper_left3_to_gripper_left1" type="revolute">
@@ -487,5 +487,5 @@
 		<origin xyz= "-0.027 0.016 0" rpy = "0 0 0"/>
 		<mimic joint="gripper_controller" multiplier="-1.0" offset="0" />
-        <dynamics damping="2.0" friction="4.0"/>
+        <dynamics damping="0.01" friction="0.005"/>
 	</joint>
 	<joint name="gripper_base_to_gripper_right3" type="revolute">
@@ -496,5 +496,5 @@
 		<origin xyz= "0.012 0.005 0" rpy = "0 0 0"/>
 		<mimic joint="gripper_controller" multiplier="-1.0" offset="0" />
-        <dynamics damping="2.0" friction="4.0"/>
+        <dynamics damping="0.01" friction="0.005"/>
 	</joint>
 	<joint name="gripper_base_to_gripper_right2" type="revolute">
@@ -505,5 +505,5 @@
 		<origin xyz= "0.005 0.027 0" rpy = "0 0 0"/>
 		<mimic joint="gripper_controller" multiplier="-1.0" offset="0" />
-        <dynamics damping="2.0" friction="4.0"/>
+        <dynamics damping="0.01" friction="0.005"/>
 	</joint>
 	<joint name="gripper_right3_to_gripper_right1" type="revolute">
@@ -514,11 +514,78 @@
 		<origin xyz= "0.027 0.016 0" rpy = "0 0 0"/>
 		<mimic joint="gripper_controller" multiplier="1.0" offset="0" />
-        <dynamics damping="2.0" friction="4.0"/>
-	</joint>
-    <!-- JointStatePublisher publishes joint state information for the model -->
-    <gazebo>
-        <plugin filename="gz-sim-joint-state-publisher-system" name="gz::sim::systems::JointStatePublisher">
+        <dynamics damping="0.01" friction="0.005"/>
+	</joint>
+    <!-- JointStatePublisher publishes joint state information for the model.
+         In future versions of Gazebo, replace 'ignition-gazebo' with 'gz-sim' and
+         'ignition::gazebo' with 'gz::sim'
+    -->
+    <gazebo>
+        <plugin filename="ignition-gazebo-joint-state-publisher-system" name="ignition::gazebo::systems::JointStatePublisher">
             <topic>joint_states</topic>
         </plugin>
     </gazebo>
+    <!-- JointPositionController subscribes to target joint positions.
+         In future versions of Gazebo, replace 'ignition-gazebo' with 'gz-sim' and
+         'ignition::gazebo' with 'gz::sim'
+    -->
+    <gazebo>
+        <plugin filename="ignition-gazebo-joint-position-controller-system" name="ignition::gazebo::systems::JointPositionController">
+            <joint_name>link1_to_link2</joint_name>
+        </plugin>
+    </gazebo>
+    <gazebo>
+        <plugin filename="ignition-gazebo-joint-position-controller-system" name="ignition::gazebo::systems::JointPositionController">
+            <joint_name>link2_to_link3</joint_name>
+        </plugin>
+    </gazebo>
+    <gazebo>
+        <plugin filename="ignition-gazebo-joint-position-controller-system" name="ignition::gazebo::systems::JointPositionController">
+            <joint_name>link3_to_link4</joint_name>
+        </plugin>
+    </gazebo>
+    <gazebo>
+        <plugin filename="ignition-gazebo-joint-position-controller-system" name="ignition::gazebo::systems::JointPositionController">
+            <joint_name>link4_to_link5</joint_name>
+        </plugin>
+    </gazebo>
+    <gazebo>
+        <plugin filename="ignition-gazebo-joint-position-controller-system" name="ignition::gazebo::systems::JointPositionController">
+            <joint_name>link5_to_link6</joint_name>
+        </plugin>
+    </gazebo>
+    <gazebo>
+        <plugin filename="ignition-gazebo-joint-position-controller-system" name="ignition::gazebo::systems::JointPositionController">
+            <joint_name>link6_to_link6flange</joint_name>
+        </plugin>
+    </gazebo>
+    <gazebo>
+        <plugin filename="ignition-gazebo-joint-position-controller-system" name="ignition::gazebo::systems::JointPositionController">
+            <joint_name>gripper_controller</joint_name>
+        </plugin>
+    </gazebo>
+    <gazebo>
+        <plugin filename="ignition-gazebo-joint-position-controller-system" name="ignition::gazebo::systems::JointPositionController">
+            <joint_name>gripper_base_to_gripper_left2</joint_name>
+        </plugin>
+    </gazebo>
+    <gazebo>
+        <plugin filename="ignition-gazebo-joint-position-controller-system" name="ignition::gazebo::systems::JointPositionController">
+            <joint_name>gripper_left3_to_gripper_left1</joint_name>
+        </plugin>
+    </gazebo>
+    <gazebo>
+        <plugin filename="ignition-gazebo-joint-position-controller-system" name="ignition::gazebo::systems::JointPositionController">
+            <joint_name>gripper_base_to_gripper_right3</joint_name>
+        </plugin>
+    </gazebo>
+    <gazebo>
+        <plugin filename="ignition-gazebo-joint-position-controller-system" name="ignition::gazebo::systems::JointPositionController">
+            <joint_name>gripper_base_to_gripper_right2</joint_name>
+        </plugin>
+    </gazebo>
+    <gazebo>
+        <plugin filename="ignition-gazebo-joint-position-controller-system" name="ignition::gazebo::systems::JointPositionController">
+            <joint_name>gripper_right3_to_gripper_right1</joint_name>
+        </plugin>
+    </gazebo>
 </robot>
