Commit message: Modified joint position publisher to do linear interpolation

File: mycobot_gazebo/urdf/mycobot_280_gazebo.urdf.xacro (robot description, xacro)
@@ -421,5 +421,5 @@
 		<child link="link3"/>
 		<origin xyz= "0 0 -0.001" rpy = "0 ${pi/2} ${-pi/2}"/>
-        <dynamics damping="0.205" friction="0.515"/>
+        <dynamics damping="0.205" friction="0.15"/>
 	</joint>
 	<joint name="link3_to_link4" type="revolute">

Commit message: Updated launch file for Gazebo for mycobot

File: mycobot_gazebo/urdf/mycobot_280_gazebo.urdf.xacro (robot description, xacro)
@@ -1,31 +1,8 @@
 <?xml version="1.0" ?>
 <robot xmlns:xacro="http://wiki.ros.org/xacro" name="mycobot_280">
-	<!--
-		xml:
-			Declare this file as an XML document and specifies the XML version.
-		robot:
-			The root element 'robot' defines a robot model. Everything about the
-			robot configuration will be nested inside this element.
-		xmlns:xacro:
-			Declares the XML namespace for xacro, which is a XML macro language used
-			in ROS (Robot Operating System) for parameterizing XML documents.
-		name:
-			Specify the name of the robot.
-	-->
-	<!-- Reference Files: https://github.com/elephantrobotics/mycobot_ros/ -->
-	<!-- Provide a global reference frame for the robotic arm in simulation (Gazebo)
-		or visualization (RViz) environments
-	-->
 	<link name="world"/>
-	<!-- ****************** ROBOT CONSTANTS *******************************  -->
-	<!-- Source: https://www.elephantrobotics.com/en/mycobot280-for-arduino-specifications-en/ -->
-	<!-- Numbers are estimated when necessary -->
 	<xacro:property name="effort" value="5.0"/>
 	<xacro:property name="velocity" value="2.792527"/>
-	<!-- ********** LINKS ********** -->
-    <!-- Define the base plate of the robotic arm -->
 	<link name="base_link">
-		<!-- The inertial values below were taken from link1 (with slight modification.
-		They are just placeholder values. -->
 		<inertial>
 			<origin xyz="0 0 0.0" rpy="0 0 0"/>
@@ -49,17 +26,8 @@
 		</collision>
 	</link>
-	<!--Define the first link of the robotic arm. Each link represents a solid part of the robot.-->
 	<link name="link1">
-		<!--Define the inertial properties of the link, which characterizes the link's resistance
-		to changes in its rotational motion.-->
-		<inertial>
-			<!--Specify the pose of the center of mass of the link relative
-			to this link's coordinate frame.-->
-			<origin xyz="0 0 0.0" rpy="0 0 0"/>
-			<!--The mass of the link in kilograms-->
+		<inertial>
+			<origin xyz="0 0 0.0" rpy="0 0 0"/>
 			<mass value="0.12"/>
-			<!--The rotational inertia values, which reflect how easily the link can rotate around
-			different axes given the distribution of mass within the link. Here we see rotation is
-			most difficult around the y axis.-->
 			<inertia
 				ixx="0.000148" ixy="0.0" ixz="0.0"
@@ -67,18 +35,10 @@
 				izz="0.000096"/>
 		</inertial>
-		<!--Define the visual representation of the link in simulation.-->
-		<visual>
-			<!--Define the shape of the link-->
-			<geometry>
-				<!--Specify the link's visual appearance using the 3D mesh file.-->
+		<visual>
+			<geometry>
 				<mesh filename="file://$(find mycobot_description)/meshes/mycobot_280/link1.dae"/>
 			</geometry>
-			<!--Define the position and orientation of the visual representation relative to the
-			link's reference frame. Here, it's rotated by -1.5708 radians (or -90 degrees)
-			around the Z-axis.-->
 			<origin xyz = "0.0 0 0 " rpy = " 0 0 ${-pi/2}"/>
 		</visual>
-		<!--Define the shape used for collision detection during simulation. This piece is important
-		for accurate physical interactions between robot components and the environment or other objects.-->
 		<collision>
 			<geometry>
@@ -88,5 +48,4 @@
 		</collision>
 	</link>
-	<!-- Define the second link of the robotic arm, and so on.-->
 	<link name="link2">
 		<inertial>
@@ -375,6 +334,4 @@
 		</collision>
 	</link>
-	<!-- ********** JOINTS ********** -->
-	<!-- Attach the robot base to the world frame with no initial offset or rotation. -->
 	<joint name="virtual_joint" type="fixed">
 		<parent link="world"/>
@@ -382,6 +339,4 @@
 		<origin xyz= "0 0 0" rpy = "0 0 0"/>
 	</joint>
-	<!-- Define the joint name and its type as "fixed". A fixed joint
-	means the two connected links cannot move relative to each other. -->
         <joint name="base_link_to_link1" type="fixed">
             <parent link="base_link"/>
@@ -450,7 +405,4 @@
         <dynamics damping="0.01" friction="0.005"/>
 	</joint>
-	<!-- The mimic element means this joint will follow the movements of the
-		gripper_controller joint.
-	-->
 	<joint name="gripper_base_to_gripper_left2" type="revolute">
 		<axis xyz="0 0 1"/>
@@ -498,8 +450,4 @@
         <dynamics damping="0.01" friction="0.005"/>
 	</joint>
-    <!-- JointStatePublisher publishes joint state information for the model.
-         In future versions of Gazebo, replace 'ignition-gazebo' with 'gz-sim' and
-         'ignition::gazebo' with 'gz::sim'
-    -->
     <gazebo>
         <plugin filename="ignition-gazebo-joint-state-publisher-system" name="ignition::gazebo::systems::JointStatePublisher">
@@ -507,8 +455,4 @@
         </plugin>
     </gazebo>
-    <!-- JointPositionController subscribes to target joint positions.
-         In future versions of Gazebo, replace 'ignition-gazebo' with 'gz-sim' and
-         'ignition::gazebo' with 'gz::sim'
-    -->
     <gazebo>
         <plugin filename="ignition-gazebo-joint-position-controller-system" name="ignition::gazebo::systems::JointPositionController">
