Commit message: Add ROS 2 Control yaml

File: mycobot_gazebo/urdf/ros2_control/classic_gazebo/mycobot_280.urdf.xacro (robot description, xacro)
@@ -1,25 +1,9 @@
 <?xml version="1.0" ?>
 <robot xmlns:xacro="http://wiki.ros.org/xacro" name="mycobot_280">
-	<!--
-		xml:
-			Declare this file as an XML document and specifies the XML version.
-		robot:
-			The root element 'robot' defines a robot model. Everything about the
-			robot configuration will be nested inside this element.
-		xmlns:xacro:
-			Declares the XML namespace for xacro, which is a XML macro language used
-			in ROS (Robot Operating System) for parameterizing XML documents.
-		name:
-			Specify the name of the robot.
-	-->
     <xacro:include filename="$(find mycobot_gazebo)/urdf/ros2_control/classic_gazebo/mycobot_280_classic_gazebo.xacro"/>
     <xacro:include filename="$(find mycobot_gazebo)/urdf/ros2_control/classic_gazebo/mycobot_280_ros2_control.xacro"/>
-	<!-- ****************** ROBOT CONSTANTS *******************************  -->
-	<!-- Source: https://www.elephantrobotics.com/en/mycobot280-for-arduino-specifications-en/ -->
-	<!-- Numbers are estimated when necessary -->
-	<!-- Reference Files: https://github.com/elephantrobotics/mycobot_ros/ -->
+	<link name="world"/>
 	<xacro:property name="effort" value="5.0"/>
 	<xacro:property name="velocity" value="2.792527"/>
-    <!-- Transmission defines how actuators are mechanically connected to joints. -->
     <xacro:macro name="default_transmission" params="joint_name">
         <transmission name="transmission_${joint_name}">
@@ -31,12 +15,4 @@
         </transmission>
     </xacro:macro>
-	<!-- ********** LINKS ********** -->
-	<!-- Provide a global reference frame for the robotic arm in simulation (Gazebo)
-		or visualization (RViz) environments
-	-->
-	<link name="world"/>
-    <!-- Define the base plate of the robotic arm
-    	The inertial values below were taken from link1 (with slight modification.
-		They are just placeholder values. -->
 	<link name="base_link">
 		<inertial>
@@ -61,5 +37,4 @@
 		</collision>
 	</link>
-	<!--Define the first link of the robotic arm. Each link represents a solid part of the robot.-->
 	<link name="link1">
 		<inertial>
@@ -84,5 +59,4 @@
 		</collision>
 	</link>
-	<!-- Define the second link of the robotic arm, and so on.-->
 	<link name="link2">
 		<inertial>
@@ -371,5 +345,4 @@
 		</collision>
 	</link>
-    <!-- ********** COLORS ********** -->
     <gazebo reference="base_link">
         <material>Gazebo/Grey</material>
@@ -399,6 +372,4 @@
         <material>Gazebo/White</material>
     </gazebo>
-	<!-- ********** JOINTS ********** -->
-	<!-- Attach the robot base to the world frame with no initial offset or rotation. -->
 	<joint name="virtual_joint" type="fixed">
 		<parent link="world"/>
@@ -406,10 +377,8 @@
 		<origin xyz= "0 0 0" rpy = "0 0 0"/>
 	</joint>
-	<!-- Define the joint name and its type as "fixed". A fixed joint
-	means the two connected links cannot move relative to each other. -->
     <joint name="base_link_to_link1" type="fixed">
         <parent link="base_link"/>
-        <child link="link1"/>
-        <origin xyz="0 0 0" rpy="0 0 0"/>
+            <child link="link1"/>
+            <origin xyz="0 0 0" rpy="0 0 0"/>
     </joint>
 	<joint name="link1_to_link2" type="revolute">
@@ -474,7 +443,4 @@
         <dynamics damping="2.0" friction="4.0"/>
 	</joint>
-	<!-- The mimic element means this joint will follow the movements of the
-		gripper_controller joint.
-	-->
 	<joint name="gripper_base_to_gripper_left2" type="revolute">
 		<axis xyz="0 0 1"/>
@@ -522,5 +488,4 @@
         <dynamics damping="2.0" friction="4.0"/>
 	</joint>
-    <!-- Put this at the bottom of the URDF -->
     <xacro:default_transmission joint_name="link1_to_link2"/>
     <xacro:default_transmission joint_name="link2_to_link3"/>

File: mycobot_gazebo/urdf/ros2_control/classic_gazebo/mycobot_280_classic_gazebo.xacro (robot description, xacro)
@@ -4,7 +4,5 @@
     <gazebo>
         <plugin filename="libgazebo_ros2_control.so" name="gazebo_ros2_control">
-            <robot_param>robot_description</robot_param>
-            <robot_param_node>robot_state_publisher</robot_param_node>
-            <parameters></parameters>
+            <parameters>$(find mycobot_gazebo)/config/mycobot_280_controllers.yaml</parameters>
         </plugin>
     </gazebo>
