Commit message: Changes to my cobot 280 URDF

File: mycobot_description/urdf/mycobot_280_urdf.xacro (robot description, xacro)
@@ -35,5 +35,5 @@
 				<mesh filename="package://mycobot_description/meshes/mycobot_280/base_link.dae"/>
 			</geometry>
-			<origin xyz = "0.0 0 -0.03" rpy = "0 0 1.5708"/>
+			<origin xyz = "0.0 0 -0.03" rpy = "0 0 ${pi/2}"/>
 		</visual>
 		<collision>
@@ -41,5 +41,5 @@
 				<mesh filename="package://mycobot_description/meshes/mycobot_280/base_link.dae"/>
 			</geometry>
-			<origin xyz = "0.0 0 -0.03" rpy = "0 0 1.5708"/>
+			<origin xyz = "0.0 0 -0.03" rpy = "0 0 ${pi/2}"/>
 		</collision>
 	</link>
@@ -72,5 +72,5 @@
 			link's reference frame. Here, it's rotated by -1.5708 radians (or -90 degrees)
 			around the Z-axis.-->
-			<origin xyz = "0.0 0 0 " rpy = " 0 0 -1.5708"/>
+			<origin xyz = "0.0 0 0 " rpy = " 0 0 ${-pi/2}"/>
 		</visual>
 		<!--Define the shape used for collision detection during simulation. This piece is important
@@ -80,5 +80,5 @@
 				<mesh filename="package://mycobot_description/meshes/mycobot_280/link1.dae"/>
 			</geometry>
-			<origin xyz = "0.0 0 0.0 " rpy = " 0 0 -1.5708"/>
+			<origin xyz = "0.0 0 0.0 " rpy = " 0 0 ${-pi/2}"/>
 		</collision>
 	</link>
@@ -97,5 +97,5 @@
 				<mesh filename="package://mycobot_description/meshes/mycobot_280/link2.dae"/>
 			</geometry>
-			<origin xyz = "0.0 0 -0.06096" rpy = " 0 0 -1.5708"/>
+			<origin xyz = "0.0 0 -0.06096" rpy = " 0 0 ${-pi/2}"/>
 		</visual>
 		<collision>
@@ -103,5 +103,5 @@
 				<mesh filename="package://mycobot_description/meshes/mycobot_280/link2.dae"/>
 			</geometry>
-			<origin xyz = "0.0 0 -0.06096" rpy = " 0 0 -1.5708"/>
+			<origin xyz = "0.0 0 -0.06096" rpy = " 0 0 ${-pi/2}"/>
 		</collision>
 	</link>
@@ -119,5 +119,5 @@
 		   		<mesh filename="package://mycobot_description/meshes/mycobot_280/link3.dae"/>
 		  	</geometry>
-			<origin xyz = "0.0 0 0.03256 " rpy = " 0 -1.5708 0"/>
+			<origin xyz = "0.0 0 0.03256 " rpy = " 0 ${-pi/2} 0"/>
 		</visual>
 		<collision>
@@ -125,5 +125,5 @@
 		   		<mesh filename="package://mycobot_description/meshes/mycobot_280/link3.dae"/>
 		  	</geometry>
-		  	<origin xyz = "0.00 0 0.03256 " rpy = " 0 -1.5708 0"/>
+		  	<origin xyz = "0.00 0 0.03256 " rpy = " 0 ${-pi/2} 0"/>
 		</collision>
 	</link>
@@ -141,5 +141,5 @@
 				<mesh filename="package://mycobot_description/meshes/mycobot_280/link4.dae"/>
 			</geometry>
-			<origin xyz = "0.0 0 0.03056 " rpy = " 0 -1.5708 0"/>
+			<origin xyz = "0.0 0 0.03056 " rpy = " 0 ${-pi/2} 0"/>
 		</visual>
 		<collision>
@@ -147,5 +147,5 @@
 				<mesh filename="package://mycobot_description/meshes/mycobot_280/link4.dae"/>
 			</geometry>
-			<origin xyz = "-0.0 0 0.03056 " rpy = " 0 -1.5708 0"/>
+			<origin xyz = "-0.0 0 0.03056 " rpy = " 0 ${-pi/2} 0"/>
 		</collision>
 	</link>
@@ -163,5 +163,5 @@
 				<mesh filename="package://mycobot_description/meshes/mycobot_280/link5.dae"/>
 		  	</geometry>
-		  	<origin xyz = "0.0 0 -0.03356 " rpy = "-1.5708 0 0"/>
+		  	<origin xyz = "0.0 0 -0.03356 " rpy = "${-pi/2} 0 0"/>
 		</visual>
 		<collision>
@@ -169,5 +169,5 @@
 		   		<mesh filename="package://mycobot_description/meshes/mycobot_280/link5.dae"/>
 		  	</geometry>
-		  	<origin xyz = "0.0 0 -0.03356 " rpy = "-1.5708 0 0"/>
+		  	<origin xyz = "0.0 0 -0.03356 " rpy = "${-pi/2} 0 0"/>
 		</collision>
 	</link>
@@ -388,5 +388,5 @@
 			velocity: Maximum allowed angular velocity (ignored for fixed joints)
 		-->
-		<limit effort = "1000.0" lower = "-3.14" upper = "3.14159" velocity = "0"/>
+		<limit effort = "1000.0" lower = "${-pi}" upper = "${pi}" velocity = "0"/>
 		<!-- The link this joint connects to on one side -->
 		<parent link="base_link"/>
@@ -407,5 +407,5 @@
 		<parent link="link1"/>
 		<child link="link2"/>
-		<origin xyz= "0 0 0.13156" rpy = "0 0 1.5708"/>
+		<origin xyz= "0 0 0.13156" rpy = "0 0 ${pi/2}"/>
 	</joint>
 	<joint name="link2_to_link3" type="revolute">
@@ -414,5 +414,5 @@
 		<parent link="link2"/>
 		<child link="link3"/>
-		<origin xyz= "0 0 -0.001" rpy = "0 1.5708 -1.5708"/>
+		<origin xyz= "0 0 -0.001" rpy = "0 ${pi/2} ${-pi/2}"/>
 	</joint>
 	<joint name="link3_to_link4" type="revolute">
@@ -428,5 +428,5 @@
 		<parent link="link4"/>
 		<child link="link5"/>
-		<origin xyz= "-0.096 0 0.06062" rpy = "0 0 -1.5708"/>
+		<origin xyz= "-0.096 0 0.06062" rpy = "0 0 ${-pi/2}"/>
 	</joint>
 	<joint name="link5_to_link6" type="revolute">
@@ -435,5 +435,5 @@
 		<parent link="link5"/>
 		<child link="link6"/>
-		<origin xyz= "0 -0.07318 0" rpy = "1.5708 -1.5708 0"/>
+		<origin xyz= "0 -0.07318 0" rpy = "${pi/2} ${-pi/2} 0"/>
 	</joint>
 	<joint name="link6_to_link6flange" type="revolute">
@@ -442,5 +442,5 @@
 		<parent link="link6"/>
 		<child link="link6_flange"/>
-		<origin xyz= "0 0.0456 0" rpy = "-1.5708 0 0"/>
+		<origin xyz= "0 0.0456 0" rpy = "${-pi/2} 0 0"/>
 	</joint>
 	<joint name="link6flange_to_gripper_base" type="fixed">

Commit message: Tweak inertial properties in myCobot280 Xacro file

File: mycobot_description/urdf/mycobot_280_urdf.xacro (robot description, xacro)
@@ -18,4 +18,9 @@
 	-->
 	<link name="world"/>
+	<!-- ****************** ROBOT CONSTANTS *******************************  -->
+	<!-- Source: https://www.elephantrobotics.com/en/mycobot280-for-arduino-specifications-en/ -->
+	<!-- Numbers are estimated when necessary -->
+	<xacro:property name="effort" value="5.0"/>
+	<xacro:property name="velocity" value="2.792527"/>
 	<!-- ********** LINKS ********** -->
     <!-- Define the base plate of the robotic arm -->
@@ -24,10 +29,10 @@
 		They are just placeholder values. -->
 		<inertial>
-			<origin xyz="0 0 0.1" rpy="0 0 0"/>
-			<mass value="12"/>
-			<inertia
-				ixx="0.0" ixy="0.0" ixz="0.0"
-				iyy="0.5" iyz="0.0"
-				izz="0.0"/>
+			<origin xyz="0 0 0.0" rpy="0 0 0"/>
+			<mass value="0.33"/>
+			<inertia
+				ixx="0.000784" ixy="0.0" ixz="0.0"
+				iyy="0.000867" iyz="0.0"
+				izz="0.001598"/>
 		</inertial>
 		<visual>
@@ -51,14 +56,14 @@
 			<!--Specify the pose of the center of mass of the link relative
 			to this link's coordinate frame.-->
-			<origin xyz="0 0 0.1" rpy="0 0 0"/>
-			<!--The mass of the link is 10 kilograms-->
-			<mass value="10"/>
+			<origin xyz="0 0 0.0" rpy="0 0 0"/>
+			<!--The mass of the link in kilograms-->
+			<mass value="0.12"/>
 			<!--The rotational inertia values, which reflect how easily the link can rotate around
 			different axes given the distribution of mass within the link. Here we see rotation is
 			most difficult around the y axis.-->
 			<inertia
-				ixx="0.0" ixy="0.0" ixz="0.0"
-				iyy="0.5" iyz="0.0"
-				izz="0.0"/>
+				ixx="0.000148" ixy="0.0" ixz="0.0"
+				iyy="0.000148" iyz="0.0"
+				izz="0.000096"/>
 		</inertial>
 		<!--Define the visual representation of the link in simulation.-->
@@ -86,10 +91,10 @@
 	<link name="link2">
 		<inertial>
-			<origin xyz="0 0 0.1" rpy="0 0 0"/>
-			<mass value="0.2"/>
-			<inertia
-				ixx="0.0" ixy="0.0" ixz="0.0"
-				iyy="0.5" iyz="0.0"
-				izz="0.0"/>
+			<origin xyz="0 0 0.0" rpy="0 0 0"/>
+			<mass value="0.19"/>
+			<inertia
+				ixx="0.000148" ixy="0.0" ixz="0.0"
+				iyy="0.000148" iyz="0.0"
+				izz="0.000096"/>
 		</inertial>
 		<visual>
@@ -108,10 +113,10 @@
 	<link name="link3">
 		<inertial>
-			<origin xyz="0 0 0.1" rpy="0 0 0"/>
-		  	<mass value="0.2"/>
-		  	<inertia
-				ixx="0.0" ixy="0.0" ixz="0.0"
-				iyy="0.5" iyz="0.0"
-				izz="0.0"/>
+			<origin xyz="0 0 0.0" rpy="0 0 0"/>
+		  	<mass value="0.16"/>
+			<inertia
+			  ixx="0.000148" ixy="0.0" ixz="0.0"
+			  iyy="0.000148" iyz="0.0"
+			  izz="0.000096"/>
 		</inertial>
 		<visual>
@@ -130,10 +135,10 @@
 	<link name="link4">
 		<inertial>
-		  	<origin xyz="0 0 0.1" rpy="0 0 0"/>
-			<mass value="0.2"/>
-			<inertia
-			  	ixx="0.0" ixy="0.0" ixz="0.0"
-			  	iyy="0.5" iyz="0.0"
-			  	izz="0.0"/>
+		  	<origin xyz="0 0 0.0" rpy="0 0 0"/>
+			<mass value="0.124"/>
+			<inertia
+			  	ixx="0.000103" ixy="0.0" ixz="0.0"
+			  	iyy="0.000103" iyz="0.0"
+			  	izz="0.000096"/>
 		</inertial>
 		<visual>
@@ -147,15 +152,15 @@
 				<mesh filename="package://mycobot_description/meshes/mycobot_280/link4.dae"/>
 			</geometry>
-			<origin xyz = "-0.0 0 0.03056 " rpy = " 0 ${-pi/2} 0"/>
+			<origin xyz = "0.0 0 0.03056 " rpy = " 0 ${-pi/2} 0"/>
 		</collision>
 	</link>
 	<link name="link5">
 		<inertial>
-			<origin xyz="0 0 0.1" rpy="0 0 0"/>
-		  	<mass value="0.2"/>
-		  	<inertia
-				ixx="0.0" ixy="0.0" ixz="0.0"
-				iyy="0.5" iyz="0.0"
-				izz="0.0"/>
+			<origin xyz="0 0 0.0" rpy="0 0 0"/>
+		  	<mass value="0.11"/>
+			<inertia
+			  ixx="0.000103" ixy="0.0" ixz="0.0"
+			  iyy="0.000103" iyz="0.0"
+			  izz="0.000096"/>
 		</inertial>
 		<visual>
@@ -174,10 +179,10 @@
 	<link name="link6">
 		<inertial>
-			<origin xyz="0 0 0.1" rpy="0 0 0"/>
-		  	<mass value="0.2"/>
-		  	<inertia
-				ixx="0.0" ixy="0.0" ixz="0.0"
-				iyy="0.5" iyz="0.0"
-				izz="0.0"/>
+			<origin xyz="0 0 0.0" rpy="0 0 0"/>
+		  	<mass value="0.0739"/>
+			<inertia
+			  ixx="0.00006649" ixy="0.0" ixz="0.0"
+			  iyy="0.00006649" iyz="0.0"
+			  izz="0.000096"/>
 		</inertial>
 		<visual>
@@ -196,10 +201,10 @@
 	<link name="link6_flange">
 		<inertial>
-			<origin xyz="0 0 0.1" rpy="0 0 0"/>
-		  	<mass value="0.1"/>
-		  	<inertia
-				ixx="0.0" ixy="0.0" ixz="0.0"
-				iyy="0.0" iyz="0.0"
-				izz="0.0"/>
+			<origin xyz="0 0 0.0" rpy="0 0 0"/>
+		  	<mass value="0.035"/>
+		  	<inertia
+				ixx="0.0000149" ixy="0.0" ixz="0.0"
+				iyy="0.0000149" iyz="0.0"
+				izz="0.0000196"/>
 		</inertial>
 		<visual>
@@ -218,10 +223,10 @@
 	<link name="gripper_base">
 		<inertial>
-			<origin xyz="0 0 0.1" rpy="0 0 0"/>
+			<origin xyz="0 0 0.0" rpy="0 0 0"/>
 		  	<mass value="0.07"/>
 		  	<inertia
-				ixx="0.0" ixy="0.0" ixz="0.0"
-				iyy="0.0" iyz="0.0"
-				izz="0.0"/>
+				ixx="0.000010725" ixy="0.0" ixz="0.0"
+				iyy="0.000014392" iyz="0.0"
+				izz="0.000018517"/>
 		</inertial>
 		<visual>
@@ -240,10 +245,10 @@
 	<link name="gripper_left1">
 		<inertial>
-			<origin xyz="0 0 0.1" rpy="0 0 0"/>
+			<origin xyz="0 0 0.0" rpy="0 0 0"/>
 		  	<mass value="0.007"/>
 		  	<inertia
-				ixx="0.0" ixy="0.0" ixz="0.0"
-				iyy="0.0" iyz="0.0"
-				izz="0.0"/>
+				ixx="1e-6" ixy="0.0" ixz="0.0"
+				iyy="1e-6" iyz="0.0"
+				izz="1e-6"/>
 		</inertial>
 		<visual>
@@ -257,81 +262,81 @@
 		   		<mesh filename="package://mycobot_description/meshes/mycobot_280/gripper_left1.dae"/>
 		  	</geometry>
+			<origin xyz = "0.039 -0.0133 -0.012 " rpy = " 0 0 0"/>
+		</collision>
+	</link>
+	<link name="gripper_left2">
+		<inertial>
+			<origin xyz="0 0 0.0" rpy="0 0 0"/>
+		  	<mass value="0.007"/>
+		  	<inertia
+				ixx="1e-6" ixy="0.0" ixz="0.0"
+				iyy="1e-6" iyz="0.0"
+				izz="1e-6"/>
+		</inertial>
+		<visual>
+		  	<geometry>
+		   		<mesh filename="package://mycobot_description/meshes/mycobot_280/gripper_left2.dae"/>
+		  	</geometry>
+			<origin xyz = "0.005 -0.0195 -0.012 " rpy = " 0 0 0"/>
+		</visual>
+		<collision>
+		  	<geometry>
+		   		<mesh filename="package://mycobot_description/meshes/mycobot_280/gripper_left2.dae"/>
+		  	</geometry>
+				<origin xyz = "0.005 -0.0195 -0.012 " rpy = " 0 0 0"/>
+		</collision>
+	</link>
+	<link name="gripper_left3">
+		<inertial>
+			<origin xyz="0 0 0.0" rpy="0 0 0"/>
+		  	<mass value="0.007"/>
+		  	<inertia
+				ixx="1e-6" ixy="0.0" ixz="0.0"
+				iyy="1e-6" iyz="0.0"
+				izz="1e-6"/>
+		</inertial>
+		<visual>
+		  	<geometry>
+		   		<mesh filename="package://mycobot_description/meshes/mycobot_280/gripper_left3.dae"/>
+		  	</geometry>
+		<origin xyz = "0.012 0.0025 -0.012 " rpy = " 0 0 0"/>
+		</visual>
+		<collision>
+		  	<geometry>
+		   		<mesh filename="package://mycobot_description/meshes/mycobot_280/gripper_left3.dae"/>
+		  	</geometry>
+			<origin xyz = "0.012 0.0025 -0.012" rpy = " 0 0 0"/>
+		</collision>
+	</link>
+	<link name="gripper_right1">
+		<inertial>
+			<origin xyz="0 0 0.0" rpy="0 0 0"/>
+		  	<mass value="0.007"/>
+		  	<inertia
+				ixx="1e-6" ixy="0.0" ixz="0.0"
+				iyy="1e-6" iyz="0.0"
+				izz="1e-6"/>
+		</inertial>
+		<visual>
+			<geometry>
+		   		<mesh filename="package://mycobot_description/meshes/mycobot_280/gripper_right1.dae"/>
+		  	</geometry>
 			<origin xyz = "-0.039 -0.0133 -0.012 " rpy = " 0 0 0"/>
-		</collision>
-	</link>
-	<link name="gripper_left2">
-		<inertial>
-			<origin xyz="0 0 0.1" rpy="0 0 0"/>
+		</visual>
+		<collision>
+		  	<geometry>
+		   		<mesh filename="package://mycobot_description/meshes/mycobot_280/gripper_right1.dae"/>
+		  	</geometry>
+			<origin xyz = "-0.039 -0.0133 -0.012 " rpy = " 0 0 0"/>
+		</collision>
+	</link>
+	<link name="gripper_right2">
+		<inertial>
+			<origin xyz="0 0 0.0" rpy="0 0 0"/>
 		  	<mass value="0.007"/>
 		  	<inertia
-				ixx="0.0" ixy="0.0" ixz="0.0"
-				iyy="0.0" iyz="0.0"
-				izz="0.0"/>
-		</inertial>
-		<visual>
-		  	<geometry>
-		   		<mesh filename="package://mycobot_description/meshes/mycobot_280/gripper_left2.dae"/>
-		  	</geometry>
-			<origin xyz = "0.005 -0.0195 -0.012 " rpy = " 0 0 0"/>
-		</visual>
-		<collision>
-		  	<geometry>
-		   		<mesh filename="package://mycobot_description/meshes/mycobot_280/gripper_left2.dae"/>
-		  	</geometry>
-				<origin xyz = "-0.005 -0.0195 -0.012 " rpy = " 0 0 0"/>
-		</collision>
-	</link>
-	<link name="gripper_left3">
-		<inertial>
-			<origin xyz="0 0 0.1" rpy="0 0 0"/>
-		  	<mass value="0.007"/>
-		  	<inertia
-				ixx="0.0" ixy="0.0" ixz="0.0"
-				iyy="0.0" iyz="0.0"
-				izz="0.0"/>
-		</inertial>
-		<visual>
-		  	<geometry>
-		   		<mesh filename="package://mycobot_description/meshes/mycobot_280/gripper_left3.dae"/>
-		  	</geometry>
-		<origin xyz = "0.012 0.0025 -0.012 " rpy = " 0 0 0"/>
-		</visual>
-		<collision>
-		  	<geometry>
-		   		<mesh filename="package://mycobot_description/meshes/mycobot_280/gripper_left3.dae"/>
-		  	</geometry>
-			<origin xyz = "0.012 0.0025 -0.012" rpy = " 0 0 0"/>
-		</collision>
-	</link>
-	<link name="gripper_right1">
-		<inertial>
-			<origin xyz="0 0 0.1" rpy="0 0 0"/>
-		  	<mass value="0.007"/>
-		  	<inertia
-				ixx="0.0" ixy="0.0" ixz="0.0"
-				iyy="0.0" iyz="0.0"
-				izz="0.0"/>
-		</inertial>
-		<visual>
-			<geometry>
-		   		<mesh filename="package://mycobot_description/meshes/mycobot_280/gripper_right1.dae"/>
-		  	</geometry>
-			<origin xyz = "-0.039 -0.0133 -0.012 " rpy = " 0 0 0"/>
-		</visual>
-		<collision>
-		  	<geometry>
-		   		<mesh filename="package://mycobot_description/meshes/mycobot_280/gripper_right1.dae"/>
-		  	</geometry>
-			<origin xyz = "-0.039 -0.0133 -0.012 " rpy = " 0 0 0"/>
-		</collision>
-	</link>
-	<link name="gripper_right2">
-		<inertial>
-			<origin xyz="0 0 0.1" rpy="0 0 0"/>
-		  	<mass value="0.007"/>
-		  	<inertia
-				ixx="0.0" ixy="0.0" ixz="0.0"
-				iyy="0.0" iyz="0.0"
-				izz="0.0"/>
+				ixx="1e-6" ixy="0.0" ixz="0.0"
+				iyy="1e-6" iyz="0.0"
+				izz="1e-6"/>
 		</inertial>
 		<visual>
@@ -350,10 +355,10 @@
 	<link name="gripper_right3">
 		<inertial>
-			<origin xyz="0 0 0.1" rpy="0 0 0"/>
+			<origin xyz="0 0 0.0" rpy="0 0 0"/>
 		  	<mass value="0.007"/>
 		  	<inertia
-				ixx="0.0" ixy="0.0" ixz="0.0"
-				iyy="0.0" iyz="0.0"
-				izz="0.0"/>
+				ixx="1e-6" ixy="0.0" ixz="0.0"
+				iyy="1e-6" iyz="0.0"
+				izz="1e-6"/>
 		</inertial>
 		<visual>
@@ -386,7 +391,7 @@
 			lower: Minimum allowed angle in radians
 			upper: Maximum allowed angle in radians
-			velocity: Maximum allowed angular velocity (ignored for fixed joints)
+			velocity: Maximum allowed angular velocity in radians per second (ignored for fixed joints)
 		-->
-		<limit effort = "1000.0" lower = "${-pi}" upper = "${pi}" velocity = "0"/>
+		<limit effort = "${effort}" lower = "${-pi}" upper = "${pi}" velocity = "${velocity}"/>
 		<!-- The link this joint connects to on one side -->
 		<parent link="base_link"/>
@@ -404,5 +409,5 @@
 	<joint name="link1_to_link2" type="revolute">
 		<axis xyz="0 0 1"/>
-		<limit effort = "1000.0" lower = "-2.879793" upper = "2.879793" velocity = "0"/>
+		<limit effort = "${effort}" lower = "-2.879793" upper = "2.879793" velocity = "${velocity}"/>
 		<parent link="link1"/>
 		<child link="link2"/>
@@ -411,5 +416,5 @@
 	<joint name="link2_to_link3" type="revolute">
 		<axis xyz="0 0 1"/>
-		<limit effort = "1000.0" lower = "-2.879793" upper = "2.879793" velocity = "0"/>
+		<limit effort = "${effort}" lower = "-2.879793" upper = "2.879793" velocity = "${velocity}"/>
 		<parent link="link2"/>
 		<child link="link3"/>
@@ -418,5 +423,5 @@
 	<joint name="link3_to_link4" type="revolute">
 		<axis xyz=" 0 0 1"/>
-		<limit effort = "1000.0" lower = "-2.879793" upper = "2.879793" velocity = "0"/>
+		<limit effort = "${effort}" lower = "-2.879793" upper = "2.879793" velocity = "${velocity}"/>
 		<parent link="link3"/>
 		<child link="link4"/>
@@ -425,5 +430,5 @@
 	<joint name="link4_to_link5" type="revolute">
 		<axis xyz=" 0 0 1"/>
-		<limit effort = "1000.0" lower = "-2.879793" upper = "2.879793" velocity = "0"/>
+		<limit effort = "${effort}" lower = "-2.879793" upper = "2.879793" velocity = "${velocity}"/>
 		<parent link="link4"/>
 		<child link="link5"/>
@@ -432,5 +437,5 @@
 	<joint name="link5_to_link6" type="revolute">
 		<axis xyz=" 0 0 1"/>
-		<limit effort = "1000.0" lower = "-2.879793" upper = "2.879793" velocity = "0"/>
+		<limit effort = "${effort}" lower = "-2.879793" upper = "2.879793" velocity = "${velocity}"/>
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