Commit message: Changed mesh paths in URDF

File: mycobot_description/urdf/mycobot_280_urdf.xacro (robot description, xacro)
@@ -38,5 +38,5 @@
 		<visual>
 			<geometry>
-				<mesh filename="package://mycobot_description/meshes/mycobot_280/base_link.dae"/>
+				<mesh filename="file://$(find mycobot_description)/meshes/mycobot_280/base_link.dae"/>
 			</geometry>
 			<origin xyz = "0.0 0 -0.03" rpy = "0 0 ${pi/2}"/>
@@ -44,5 +44,5 @@
 		<collision>
 			<geometry>
-				<mesh filename="package://mycobot_description/meshes/mycobot_280/base_link.dae"/>
+				<mesh filename="file://$(find mycobot_description)/meshes/mycobot_280/base_link.dae"/>
 			</geometry>
 			<origin xyz = "0.0 0 -0.03" rpy = "0 0 ${pi/2}"/>
@@ -72,5 +72,5 @@
 			<geometry>
 				<!--Specify the link's visual appearance using the 3D mesh file.-->
-				<mesh filename="package://mycobot_description/meshes/mycobot_280/link1.dae"/>
+				<mesh filename="file://$(find mycobot_description)/meshes/mycobot_280/link1.dae"/>
 			</geometry>
 			<!--Define the position and orientation of the visual representation relative to the
@@ -83,5 +83,5 @@
 		<collision>
 			<geometry>
-				<mesh filename="package://mycobot_description/meshes/mycobot_280/link1.dae"/>
+				<mesh filename="file://$(find mycobot_description)/meshes/mycobot_280/link1.dae"/>
 			</geometry>
 			<origin xyz = "0.0 0 0.0 " rpy = " 0 0 ${-pi/2}"/>
@@ -100,5 +100,5 @@
 		<visual>
 			<geometry>
-				<mesh filename="package://mycobot_description/meshes/mycobot_280/link2.dae"/>
+				<mesh filename="file://$(find mycobot_description)/meshes/mycobot_280/link2.dae"/>
 			</geometry>
 			<origin xyz = "0.0 0 -0.06096" rpy = " 0 0 ${-pi/2}"/>
@@ -106,5 +106,5 @@
 		<collision>
 			<geometry>
-				<mesh filename="package://mycobot_description/meshes/mycobot_280/link2.dae"/>
+				<mesh filename="file://$(find mycobot_description)/meshes/mycobot_280/link2.dae"/>
 			</geometry>
 			<origin xyz = "0.0 0 -0.06096" rpy = " 0 0 ${-pi/2}"/>
@@ -122,5 +122,5 @@
 		<visual>
 		  	<geometry>
-		   		<mesh filename="package://mycobot_description/meshes/mycobot_280/link3.dae"/>
+		   		<mesh filename="file://$(find mycobot_description)/meshes/mycobot_280/link3.dae"/>
 		  	</geometry>
 			<origin xyz = "0.0 0 0.03256 " rpy = " 0 ${-pi/2} 0"/>
@@ -128,5 +128,5 @@
 		<collision>
 		  	<geometry>
-		   		<mesh filename="package://mycobot_description/meshes/mycobot_280/link3.dae"/>
+		   		<mesh filename="file://$(find mycobot_description)/meshes/mycobot_280/link3.dae"/>
 		  	</geometry>
 		  	<origin xyz = "0.00 0 0.03256 " rpy = " 0 ${-pi/2} 0"/>
@@ -144,5 +144,5 @@
 		<visual>
 			<geometry>
-				<mesh filename="package://mycobot_description/meshes/mycobot_280/link4.dae"/>
+				<mesh filename="file://$(find mycobot_description)/meshes/mycobot_280/link4.dae"/>
 			</geometry>
 			<origin xyz = "0.0 0 0.03056 " rpy = " 0 ${-pi/2} 0"/>
@@ -150,5 +150,5 @@
 		<collision>
 			<geometry>
-				<mesh filename="package://mycobot_description/meshes/mycobot_280/link4.dae"/>
+				<mesh filename="file://$(find mycobot_description)/meshes/mycobot_280/link4.dae"/>
 			</geometry>
 			<origin xyz = "0.0 0 0.03056 " rpy = " 0 ${-pi/2} 0"/>
@@ -166,5 +166,5 @@
 		<visual>
 		  	<geometry>
-				<mesh filename="package://mycobot_description/meshes/mycobot_280/link5.dae"/>
+				<mesh filename="file://$(find mycobot_description)/meshes/mycobot_280/link5.dae"/>
 		  	</geometry>
 		  	<origin xyz = "0.0 0 -0.03356 " rpy = "${-pi/2} 0 0"/>
@@ -172,5 +172,5 @@
 		<collision>
 		   	<geometry>
-		   		<mesh filename="package://mycobot_description/meshes/mycobot_280/link5.dae"/>
+		   		<mesh filename="file://$(find mycobot_description)/meshes/mycobot_280/link5.dae"/>
 		  	</geometry>
 		  	<origin xyz = "0.0 0 -0.03356 " rpy = "${-pi/2} 0 0"/>
@@ -188,5 +188,5 @@
 		<visual>
 		  	<geometry>
-				<mesh filename="package://mycobot_description/meshes/mycobot_280/link6.dae"/>
+				<mesh filename="file://$(find mycobot_description)/meshes/mycobot_280/link6.dae"/>
 		  	</geometry>
 		  	<origin xyz = "0 0.00 -0.038" rpy = "0 0 0"/>
@@ -194,5 +194,5 @@
 		<collision>
 		   	<geometry>
-		   		<mesh filename="package://mycobot_description/meshes/mycobot_280/link6.dae"/>
+		   		<mesh filename="file://$(find mycobot_description)/meshes/mycobot_280/link6.dae"/>
 		  	</geometry>
 		  	<origin xyz = "0 0.00 -0.038" rpy = "0 0 0"/>
@@ -210,5 +210,5 @@
 		<visual>
 		  	<geometry>
-				<mesh filename="package://mycobot_description/meshes/mycobot_280/link7.dae"/>
+				<mesh filename="file://$(find mycobot_description)/meshes/mycobot_280/link7.dae"/>
 		  	</geometry>
 		  	<origin xyz = "0.0 0 -0.012 " rpy = "0 0 0"/>
@@ -216,5 +216,5 @@
 		<collision>
 		   	<geometry>
-		   		<mesh filename="package://mycobot_description/meshes/mycobot_280/link7.dae"/>
+		   		<mesh filename="file://$(find mycobot_description)/meshes/mycobot_280/link7.dae"/>
 		  	</geometry>
 		  	<origin xyz = "0.0 0 -0.012 " rpy = "0 0 0"/>
@@ -232,5 +232,5 @@
 		<visual>
 		  	<geometry>
-				<mesh filename="package://mycobot_description/meshes/mycobot_280/gripper_base.dae"/>
+				<mesh filename="file://$(find mycobot_description)/meshes/mycobot_280/gripper_base.dae"/>
 		  	</geometry>
 		  	<origin xyz = "0.0 0.0 -0.012" rpy = "0 0 0"/>
@@ -238,5 +238,5 @@
 		<collision>
 		   	<geometry>
-		   		<mesh filename="package://mycobot_description/meshes/mycobot_280/gripper_base.dae"/>
+		   		<mesh filename="file://$(find mycobot_description)/meshes/mycobot_280/gripper_base.dae"/>
 		  	</geometry>
 		  	<origin xyz = "0.0 0.0 -0.012" rpy = "0 0 0"/>
@@ -254,5 +254,5 @@
 		<visual>
 		  	<geometry>
-		  		<mesh filename="package://mycobot_description/meshes/mycobot_280/gripper_left1.dae"/>
+		  		<mesh filename="file://$(find mycobot_description)/meshes/mycobot_280/gripper_left1.dae"/>
 		  	</geometry>
 			<origin xyz = "0.039 -0.0133 -0.012 " rpy = " 0 0 0"/>
@@ -260,5 +260,5 @@
 		<collision>
 		  	<geometry>
-		   		<mesh filename="package://mycobot_description/meshes/mycobot_280/gripper_left1.dae"/>
+		   		<mesh filename="file://$(find mycobot_description)/meshes/mycobot_280/gripper_left1.dae"/>
 		  	</geometry>
 			<origin xyz = "0.039 -0.0133 -0.012 " rpy = " 0 0 0"/>
@@ -276,5 +276,5 @@
 		<visual>
 		  	<geometry>
-		   		<mesh filename="package://mycobot_description/meshes/mycobot_280/gripper_left2.dae"/>
+		   		<mesh filename="file://$(find mycobot_description)/meshes/mycobot_280/gripper_left2.dae"/>
 		  	</geometry>
 			<origin xyz = "0.005 -0.0195 -0.012 " rpy = " 0 0 0"/>
@@ -282,5 +282,5 @@
 		<collision>
 		  	<geometry>
-		   		<mesh filename="package://mycobot_description/meshes/mycobot_280/gripper_left2.dae"/>
+		   		<mesh filename="file://$(find mycobot_description)/meshes/mycobot_280/gripper_left2.dae"/>
 		  	</geometry>
 				<origin xyz = "0.005 -0.0195 -0.012 " rpy = " 0 0 0"/>
@@ -298,5 +298,5 @@
 		<visual>
 		  	<geometry>
-		   		<mesh filename="package://mycobot_description/meshes/mycobot_280/gripper_left3.dae"/>
+		   		<mesh filename="file://$(find mycobot_description)/meshes/mycobot_280/gripper_left3.dae"/>
 		  	</geometry>
 		<origin xyz = "0.012 0.0025 -0.012 " rpy = " 0 0 0"/>
@@ -304,5 +304,5 @@
 		<collision>
 		  	<geometry>
-		   		<mesh filename="package://mycobot_description/meshes/mycobot_280/gripper_left3.dae"/>
+		   		<mesh filename="file://$(find mycobot_description)/meshes/mycobot_280/gripper_left3.dae"/>
 		  	</geometry>
 			<origin xyz = "0.012 0.0025 -0.012" rpy = " 0 0 0"/>
@@ -320,5 +320,5 @@
 		<visual>
 			<geometry>
-		   		<mesh filename="package://mycobot_description/meshes/mycobot_280/gripper_right1.dae"/>
+		   		<mesh filename="file://$(find mycobot_description)/meshes/mycobot_280/gripper_right1.dae"/>
 		  	</geometry>
 			<origin xyz = "-0.039 -0.0133 -0.012 " rpy = " 0 0 0"/>
@@ -326,5 +326,5 @@
 		<collision>
 		  	<geometry>
-		   		<mesh filename="package://mycobot_description/meshes/mycobot_280/gripper_right1.dae"/>
+		   		<mesh filename="file://$(find mycobot_description)/meshes/mycobot_280/gripper_right1.dae"/>
 		  	</geometry>
 			<origin xyz = "-0.039 -0.0133 -0.012 " rpy = " 0 0 0"/>
@@ -342,5 +342,5 @@
 		<visual>
 			<geometry>
-		   		<mesh filename="package://mycobot_description/meshes/mycobot_280/gripper_right2.dae"/>
+		   		<mesh filename="file://$(find mycobot_description)/meshes/mycobot_280/gripper_right2.dae"/>
 		 	</geometry>
 			<origin xyz = "-0.005 -0.0195 -0.012 " rpy = " 0 0 0"/>
@@ -348,5 +348,5 @@
 		<collision>
 		  	<geometry>
-		   		<mesh filename="package://mycobot_description/meshes/mycobot_280/gripper_right2.dae"/>
+		   		<mesh filename="file://$(find mycobot_description)/meshes/mycobot_280/gripper_right2.dae"/>
 		  	</geometry>
 			<origin xyz = "-0.005 -0.0195 -0.012 " rpy = " 0 0 0"/>
@@ -364,5 +364,5 @@
 		<visual>
 			<geometry>
-		   		<mesh filename="package://mycobot_description/meshes/mycobot_280/gripper_right3.dae"/>
+		   		<mesh filename="file://$(find mycobot_description)/meshes/mycobot_280/gripper_right3.dae"/>
 			</geometry>
 			<origin xyz = "-0.012 0.0025 -0.012 " rpy = " 0 0 0"/>
@@ -370,5 +370,5 @@
 		<collision>
 		  	<geometry>
-		   		<mesh filename="package://mycobot_description/meshes/mycobot_280/gripper_right3.dae"/>
+		   		<mesh filename="file://$(find mycobot_description)/meshes/mycobot_280/gripper_right3.dae"/>
 		  	</geometry>
 			<origin xyz = "-0.012 0.0025 -0.012" rpy = " 0 0 0"/>

Commit message: Improved URDF collision geometry

File: mycobot_description/urdf/mycobot_280_urdf.xacro (robot description, xacro)
@@ -44,7 +44,7 @@
 		<collision>
 			<geometry>
-				<mesh filename="file://$(find mycobot_description)/meshes/mycobot_280/base_link.dae"/>
-			</geometry>
-			<origin xyz = "0.0 0 -0.03" rpy = "0 0 ${pi/2}"/>
+				<box size="0.115 0.14 0.02"/>
+			</geometry>
+			<origin xyz = "0.0 0 -0.015" rpy = "0 0 0"/>
 		</collision>
 	</link>
@@ -83,7 +83,7 @@
 		<collision>
 			<geometry>
-				<mesh filename="file://$(find mycobot_description)/meshes/mycobot_280/link1.dae"/>
-			</geometry>
-			<origin xyz = "0.0 0 0.0 " rpy = " 0 0 ${-pi/2}"/>
+			     <box size="0.08 0.12 0.075"/>
+			</geometry>
+			<origin xyz = "0.0 -0.01 0.034" rpy = " 0 0 0"/>
 		</collision>
 	</link>
@@ -106,7 +106,7 @@
 		<collision>
 			<geometry>
-				<mesh filename="file://$(find mycobot_description)/meshes/mycobot_280/link2.dae"/>
-			</geometry>
-			<origin xyz = "0.0 0 -0.06096" rpy = " 0 0 ${-pi/2}"/>
+				<cylinder radius="0.025" length="0.085"/>
+			</geometry>
+			<origin xyz = "0.0 0 -0.02" rpy = " 0 0 ${-pi/2}"/>
 		</collision>
 	</link>
@@ -127,8 +127,8 @@
 		</visual>
 		<collision>
-		  	<geometry>
-		   		<mesh filename="file://$(find mycobot_description)/meshes/mycobot_280/link3.dae"/>
-		  	</geometry>
-		  	<origin xyz = "0.00 0 0.03256 " rpy = " 0 ${-pi/2} 0"/>
+			<geometry>
+				<cylinder radius="0.025" length="0.15"/>
+			</geometry>
+			<origin xyz = "-0.058 0 0.059" rpy = "0 ${-pi/2} 0"/>
 		</collision>
 	</link>
@@ -150,7 +150,7 @@
 		<collision>
 			<geometry>
-				<mesh filename="file://$(find mycobot_description)/meshes/mycobot_280/link4.dae"/>
-			</geometry>
-			<origin xyz = "0.0 0 0.03056 " rpy = " 0 ${-pi/2} 0"/>
+				<cylinder radius="0.025" length="0.125"/>
+			</geometry>
+			<origin xyz = "-0.05 0 0.0" rpy = "0 ${-pi/2} 0"/>
 		</collision>
 	</link>
@@ -171,8 +171,8 @@
 		</visual>
 		<collision>
-		   	<geometry>
-		   		<mesh filename="file://$(find mycobot_description)/meshes/mycobot_280/link5.dae"/>
-		  	</geometry>
-		  	<origin xyz = "0.0 0 -0.03356 " rpy = "${-pi/2} 0 0"/>
+			<geometry>
+				<box size="0.03 0.035 0.05"/>
+			</geometry>
+			<origin xyz = "0.0 0 -0.005" rpy = "0 0.0 0"/>
 		</collision>
 	</link>
@@ -194,7 +194,7 @@
 		<collision>
 		   	<geometry>
-		   		<mesh filename="file://$(find mycobot_description)/meshes/mycobot_280/link6.dae"/>
-		  	</geometry>
-		  	<origin xyz = "0 0.00 -0.038" rpy = "0 0 0"/>
+		   		<cylinder radius="0.025" length="0.06"/>
+		  	</geometry>
+		  	<origin xyz = "0 0.00 0.0" rpy = "${-pi/2} 0 0"/>
 		</collision>
 	</link>
@@ -216,7 +216,7 @@
 		<collision>
 		   	<geometry>
-		   		<mesh filename="file://$(find mycobot_description)/meshes/mycobot_280/link7.dae"/>
-		  	</geometry>
-		  	<origin xyz = "0.0 0 -0.012 " rpy = "0 0 0"/>
+		   		<cylinder radius="0.02" length="0.02"/>
+		  	</geometry>
+		  	<origin xyz = "0 0.00 0.0" rpy = "0 0 0"/>
 		</collision>
 	</link>
@@ -238,7 +238,7 @@
 		<collision>
 		   	<geometry>
-		   		<mesh filename="file://$(find mycobot_description)/meshes/mycobot_280/gripper_base.dae"/>
-		  	</geometry>
-		  	<origin xyz = "0.0 0.0 -0.012" rpy = "0 0 0"/>
+		   		<box size="0.065 0.025 0.025"/>
+		  	</geometry>
+		  	<origin xyz = "0.0 0.0 0.0" rpy = "0 0 0"/>
 		</collision>
 	</link>
@@ -260,7 +260,7 @@
 		<collision>
 		  	<geometry>
-		   		<mesh filename="file://$(find mycobot_description)/meshes/mycobot_280/gripper_left1.dae"/>
-		  	</geometry>
-			<origin xyz = "0.039 -0.0133 -0.012 " rpy = " 0 0 0"/>
+		   		<box size="0.02 0.02 0.02"/>
+		  	</geometry>
+			<origin xyz = "0.013 0.042 -0.010 " rpy = " 0 0 0"/>
 		</collision>
 	</link>
@@ -282,7 +282,7 @@
 		<collision>
 		  	<geometry>
-		   		<mesh filename="file://$(find mycobot_description)/meshes/mycobot_280/gripper_left2.dae"/>
-		  	</geometry>
-				<origin xyz = "0.005 -0.0195 -0.012 " rpy = " 0 0 0"/>
+		   		<box size="0.02 0.02 0.02"/>
+		  	</geometry>
+			<origin xyz = "-0.025 0.0 -0.010 " rpy = " 0 0 0"/>
 		</collision>
 	</link>
@@ -304,7 +304,7 @@
 		<collision>
 		  	<geometry>
-		   		<mesh filename="file://$(find mycobot_description)/meshes/mycobot_280/gripper_left3.dae"/>
-		  	</geometry>
-			<origin xyz = "0.012 0.0025 -0.012" rpy = " 0 0 0"/>
+		   		<box size="0.01 0.01 0.01"/>
+		  	</geometry>
+			<origin xyz = "-0.014 0.005 0.005 " rpy = " 0 0 0"/>
 		</collision>
 	</link>
@@ -326,7 +326,7 @@
 		<collision>
 		  	<geometry>
-		   		<mesh filename="file://$(find mycobot_description)/meshes/mycobot_280/gripper_right1.dae"/>
-		  	</geometry>
-			<origin xyz = "-0.039 -0.0133 -0.012 " rpy = " 0 0 0"/>
+		   		<box size="0.02 0.02 0.02"/>
+		  	</geometry>
+			<origin xyz = "-0.013 0.042 -0.010 " rpy = " 0 0 0"/>
 		</collision>
 	</link>
@@ -348,7 +348,7 @@
 		<collision>
 		  	<geometry>
-		   		<mesh filename="file://$(find mycobot_description)/meshes/mycobot_280/gripper_right2.dae"/>
-		  	</geometry>
-			<origin xyz = "-0.005 -0.0195 -0.012 " rpy = " 0 0 0"/>
+		   		<box size="0.02 0.02 0.02"/>
+		  	</geometry>
+			<origin xyz = "0.025 0.0 -0.010 " rpy = " 0 0 0"/>
 		</collision>
 	</link>
@@ -370,7 +370,7 @@
 		<collision>
 		  	<geometry>
-		   		<mesh filename="file://$(find mycobot_description)/meshes/mycobot_280/gripper_right3.dae"/>
-		  	</geometry>
-			<origin xyz = "-0.012 0.0025 -0.012" rpy = " 0 0 0"/>
+		   		<box size="0.01 0.01 0.01"/>
+		  	</geometry>
+			<origin xyz = "0.014 0.005 0.005 " rpy = " 0 0 0"/>
 		</collision>
 	</link>

File: mycobot_gazebo/urdf/ros2_control/gazebo/mycobot_280.urdf.xacro (robot description, xacro)
@@ -23,7 +23,7 @@
 		<collision>
 			<geometry>
-				<mesh filename="file://$(find mycobot_description)/meshes/mycobot_280/base_link.dae"/>
-			</geometry>
-			<origin xyz = "0.0 0 -0.03" rpy = "0 0 ${pi/2}"/>
+				<box size="0.115 0.14 0.02"/>
+			</geometry>
+			<origin xyz = "0.0 0 -0.015" rpy = "0 0 0"/>
 		</collision>
 	</link>
@@ -45,7 +45,7 @@
 		<collision>
 			<geometry>
-				<mesh filename="file://$(find mycobot_description)/meshes/mycobot_280/link1.dae"/>
-			</geometry>
-			<origin xyz = "0.0 0 0.0 " rpy = " 0 0 ${-pi/2}"/>
+			     <box size="0.08 0.12 0.075"/>
+			</geometry>
+			<origin xyz = "0.0 -0.01 0.034" rpy = " 0 0 0"/>
 		</collision>
 	</link>
@@ -67,7 +67,7 @@
 		<collision>
 			<geometry>
-				<mesh filename="file://$(find mycobot_description)/meshes/mycobot_280/link2.dae"/>
-			</geometry>
-			<origin xyz = "0.0 0 -0.06096" rpy = " 0 0 ${-pi/2}"/>
+				<cylinder radius="0.025" length="0.085"/>
+			</geometry>
+			<origin xyz = "0.0 0 -0.02" rpy = " 0 0 ${-pi/2}"/>
 		</collision>
 	</link>
@@ -88,8 +88,8 @@
 		</visual>
 		<collision>
-		  	<geometry>
-		   		<mesh filename="file://$(find mycobot_description)/meshes/mycobot_280/link3.dae"/>
-		  	</geometry>
-		  	<origin xyz = "0.00 0 0.03256 " rpy = " 0 ${-pi/2} 0"/>
+			<geometry>
+				<cylinder radius="0.025" length="0.15"/>
+			</geometry>
+			<origin xyz = "-0.058 0 0.059" rpy = "0 ${-pi/2} 0"/>
 		</collision>
 	</link>
@@ -111,7 +111,7 @@
 		<collision>
 			<geometry>
-				<mesh filename="file://$(find mycobot_description)/meshes/mycobot_280/link4.dae"/>
-			</geometry>
-			<origin xyz = "0.0 0 0.03056 " rpy = " 0 ${-pi/2} 0"/>
+				<cylinder radius="0.025" length="0.125"/>
+			</geometry>
+			<origin xyz = "-0.05 0 0.0" rpy = "0 ${-pi/2} 0"/>
 		</collision>
 	</link>
@@ -132,8 +132,8 @@
 		</visual>
 		<collision>
-		   	<geometry>
-		   		<mesh filename="file://$(find mycobot_description)/meshes/mycobot_280/link5.dae"/>
-		  	</geometry>
-		  	<origin xyz = "0.0 0 -0.03356 " rpy = "${-pi/2} 0 0"/>
+			<geometry>
+				<box size="0.03 0.035 0.05"/>
+			</geometry>
+			<origin xyz = "0.0 0 -0.005" rpy = "0 0.0 0"/>
 		</collision>
 	</link>
@@ -155,7 +155,7 @@
 		<collision>
 		   	<geometry>
-		   		<mesh filename="file://$(find mycobot_description)/meshes/mycobot_280/link6.dae"/>
-		  	</geometry>
-		  	<origin xyz = "0 0.00 -0.038" rpy = "0 0 0"/>
+		   		<cylinder radius="0.025" length="0.06"/>
+		  	</geometry>
+		  	<origin xyz = "0 0.00 0.0" rpy = "${-pi/2} 0 0"/>
 		</collision>
 	</link>
@@ -177,7 +177,7 @@
 		<collision>
 		   	<geometry>
-		   		<mesh filename="file://$(find mycobot_description)/meshes/mycobot_280/link7.dae"/>
-		  	</geometry>
-		  	<origin xyz = "0.0 0 -0.012 " rpy = "0 0 0"/>
+		   		<cylinder radius="0.02" length="0.02"/>
+		  	</geometry>
+		  	<origin xyz = "0 0.00 0.0" rpy = "0 0 0"/>
 		</collision>
 	</link>
@@ -199,7 +199,7 @@
 		<collision>
 		   	<geometry>
-		   		<mesh filename="file://$(find mycobot_description)/meshes/mycobot_280/gripper_base.dae"/>
-		  	</geometry>
-		  	<origin xyz = "0.0 0.0 -0.012" rpy = "0 0 0"/>
+		   		<box size="0.065 0.025 0.025"/>
+		  	</geometry>
+		  	<origin xyz = "0.0 0.0 0.0" rpy = "0 0 0"/>
 		</collision>
 	</link>
@@ -221,7 +221,7 @@
 		<collision>
 		  	<geometry>
-		   		<mesh filename="file://$(find mycobot_description)/meshes/mycobot_280/gripper_left1.dae"/>
-		  	</geometry>
-			<origin xyz = "0.039 -0.0133 -0.012 " rpy = " 0 0 0"/>
+		   		<box size="0.02 0.02 0.02"/>
+		  	</geometry>
+			<origin xyz = "0.013 0.042 -0.010 " rpy = " 0 0 0"/>
 		</collision>
 	</link>
@@ -243,7 +243,7 @@
 		<collision>
 		  	<geometry>
-		   		<mesh filename="file://$(find mycobot_description)/meshes/mycobot_280/gripper_left2.dae"/>
-		  	</geometry>
-				<origin xyz = "0.005 -0.0195 -0.012 " rpy = " 0 0 0"/>
+		   		<box size="0.02 0.02 0.02"/>
+		  	</geometry>
+			<origin xyz = "-0.025 0.0 -0.010 " rpy = " 0 0 0"/>
 		</collision>
 	</link>
@@ -265,7 +265,7 @@
 		<collision>
 		  	<geometry>
-		   		<mesh filename="file://$(find mycobot_description)/meshes/mycobot_280/gripper_left3.dae"/>
-		  	</geometry>
-			<origin xyz = "0.012 0.0025 -0.012" rpy = " 0 0 0"/>
+		   		<box size="0.01 0.01 0.01"/>
+		  	</geometry>
+			<origin xyz = "-0.014 0.005 0.005 " rpy = " 0 0 0"/>
 		</collision>
 	</link>
@@ -287,7 +287,7 @@
 		<collision>
 		  	<geometry>
-		   		<mesh filename="file://$(find mycobot_description)/meshes/mycobot_280/gripper_right1.dae"/>
-		  	</geometry>
-			<origin xyz = "-0.039 -0.0133 -0.012 " rpy = " 0 0 0"/>
+		   		<box size="0.02 0.02 0.02"/>
+		  	</geometry>
+			<origin xyz = "-0.013 0.042 -0.010 " rpy = " 0 0 0"/>
 		</collision>
 	</link>
@@ -309,7 +309,7 @@
 		<collision>
 		  	<geometry>
-		   		<mesh filename="file://$(find mycobot_description)/meshes/mycobot_280/gripper_right2.dae"/>
-		  	</geometry>
-			<origin xyz = "-0.005 -0.0195 -0.012 " rpy = " 0 0 0"/>
+		   		<box size="0.02 0.02 0.02"/>
+		  	</geometry>
+			<origin xyz = "0.025 0.0 -0.010 " rpy = " 0 0 0"/>
 		</collision>
 	</link>
@@ -331,7 +331,7 @@
 		<collision>
 		  	<geometry>
-		   		<mesh filename="file://$(find mycobot_description)/meshes/mycobot_280/gripper_right3.dae"/>
-		  	</geometry>
-			<origin xyz = "-0.012 0.0025 -0.012" rpy = " 0 0 0"/>
+		   		<box size="0.01 0.01 0.01"/>
+		  	</geometry>
+			<origin xyz = "0.014 0.005 0.005 " rpy = " 0 0 0"/>
 		</collision>
 	</link>

Commit message: Best parameters so far for pick and place

File: mycobot_description/urdf/mycobot_280_urdf.xacro (robot description, xacro)
@@ -44,5 +44,5 @@
 		<collision>
 			<geometry>
-				<box size="0.115 0.14 0.02"/>
+				<box size="0.105 0.14 0.02"/>
 			</geometry>
 			<origin xyz = "0.0 0 -0.015" rpy = "0 0 0"/>

File: mycobot_gazebo/urdf/ros2_control/gazebo/mycobot_280.urdf.xacro (robot description, xacro)
@@ -23,5 +23,5 @@
 		<collision>
 			<geometry>
-				<box size="0.115 0.14 0.02"/>
+				<box size="0.105 0.14 0.02"/>
 			</geometry>
 			<origin xyz = "0.0 0 -0.015" rpy = "0 0 0"/>

Commit message: Updated URDF for Gripper

File: mycobot_description/urdf/mycobot_280_urdf.xacro (robot description, xacro)
@@ -260,5 +260,5 @@
 		<collision>
 		  	<geometry>
-		   		<box size="0.02 0.02 0.02"/>
+		   		<box size="0.013 0.02 0.015"/>
 		  	</geometry>
 			<origin xyz = "0.013 0.042 -0.010 " rpy = " 0 0 0"/>
@@ -326,5 +326,5 @@
 		<collision>
 		  	<geometry>
-		   		<box size="0.02 0.02 0.02"/>
+		   		<box size="0.013 0.02 0.015"/>
 		  	</geometry>
 			<origin xyz = "-0.013 0.042 -0.010 " rpy = " 0 0 0"/>

File: mycobot_gazebo/urdf/ros2_control/gazebo/mycobot_280.urdf.xacro (robot description, xacro)
@@ -221,5 +221,5 @@
 		<collision>
 		  	<geometry>
-		   		<box size="0.02 0.02 0.02"/>
+		   		<box size="0.013 0.02 0.015"/>
 		  	</geometry>
 			<origin xyz = "0.013 0.042 -0.010 " rpy = " 0 0 0"/>
@@ -287,5 +287,5 @@
 		<collision>
 		  	<geometry>
-		   		<box size="0.02 0.02 0.02"/>
+		   		<box size="0.013 0.02 0.015"/>
 		  	</geometry>
 			<origin xyz = "-0.013 0.042 -0.010 " rpy = " 0 0 0"/>
