Commit message: Add depth camera holder to URDF

File: hello_mtc_with_perception/urdf/mycobot_280.urdf.xacro (robot description, xacro)
@@ -2,3 +2,75 @@
 <robot name="mycobot_280" xmlns:xacro="http://www.ros.org/wiki/xacro">
   <xacro:include filename="$(find mycobot_gazebo)/urdf/ros2_control/gazebo/mycobot_280.urdf.xacro"/>
+  <link name="torso_link">
+    <inertial>
+      <origin xyz="0 0 0.20" />
+      <mass value="2.5" />
+      <inertia ixx="0.8" ixy="0.0" ixz="0.0" iyy="0.8" iyz="0.0" izz="0.8" />
+    </inertial>
+    <visual name="holder">
+      <origin xyz="0 0 0.20" rpy="0 0 0" />
+      <material name="LightGrey">
+        <color rgba="0.7 0.7 0.7 1.0"/>
+      </material>
+      <geometry>
+        <cylinder radius="0.005" length="0.4"/>
+      </geometry>
+    </visual>
+    <visual name="base">
+      <origin xyz="0 0 0" rpy="0 0 0" />
+      <material name="LightGrey">
+        <color rgba="0.7 0.7 0.7 1.0"/>
+      </material>
+      <geometry>
+        <box size="0.15 0.10 0.04" />
+      </geometry>
+    </visual>
+    <collision name="holder">
+      <origin xyz="0 0 0.20" rpy="0 0 0" />
+      <geometry>
+        <cylinder radius="0.005" length="0.4"/>
+      </geometry>
+    </collision>
+    <collision name="base">
+      <origin xyz="0 0 0.0" rpy="0 0 0" />
+      <geometry>
+        <box size="0.15 0.10 0.04" />
+      </geometry>
+    </collision>
+  </link>
+  <joint name="base_link_to_torso_link" type="fixed">
+    <parent link="base_link"/>
+    <child link="torso_link"/>
+    <origin xyz="0.22 -0.25 0" rpy="0 0 0"/>
+  </joint>
+  <gazebo reference="torso_link">
+    <visual>
+      <material>
+        <ambient>0.7 0.7 0.7 1</ambient>
+        <diffuse>0.7 0.7 0.7 1</diffuse>
+        <specular>0.1 0.1 0.1 1</specular>
+      </material>
+    </visual>
+  </gazebo>
+  <gazebo reference="camera_head_link">
+    <sensor name="camera_head" type="rgbd_camera">
+      <topic>camera_head</topic>
+      <gz_frame_id>camera_head_link</gz_frame_id>
+      <update_rate>30</update_rate>
+      <always_on>true</always_on>
+      <visualize>true</visualize>
+      <camera>
+        <optical_frame_id>camera_head_depth_optical_frame</optical_frame_id>
+        <horizontal_fov>1.5184</horizontal_fov>
+        <image>
+          <width>424</width>
+          <height>240</height>
+        </image>
+        <clip>
+          <near>0.05</near>
+          <far>1.5</far>
+        </clip>
+      </camera>
+    </sensor>
+  </gazebo>
 </robot>

Commit message: Added STL file for Intel Realsense depth camera

File: hello_mtc_with_perception/urdf/mycobot_280.urdf.xacro (robot description, xacro)
@@ -2,4 +2,12 @@
 <robot name="mycobot_280" xmlns:xacro="http://www.ros.org/wiki/xacro">
   <xacro:include filename="$(find mycobot_gazebo)/urdf/ros2_control/gazebo/mycobot_280.urdf.xacro"/>
+  <xacro:property name="M_PI" value="3.1415926535897931" />
+  <xacro:property name="d435_cam_width" value="0.090"/>
+  <xacro:property name="d435_cam_height" value="0.025"/>
+  <xacro:property name="d435_cam_depth" value="0.02505"/>
+  <xacro:property name="d435_cam_depth_to_infra1_offset" value="0.0"/>
+  <xacro:property name="d435_cam_depth_to_infra2_offset" value="-0.050"/>
+  <xacro:property name="d435_cam_depth_to_color_offset" value="0.015"/>
+  <xacro:property name="camera_tilt_angle_deg" value="15"/>
   <link name="torso_link">
     <inertial>
@@ -44,13 +52,79 @@
     <origin xyz="0.22 -0.25 0" rpy="0 0 0"/>
   </joint>
-  <gazebo reference="torso_link">
+  <joint name="camera_head_joint" type="fixed">
+    <parent link="torso_link"/>
+    <child link="camera_head_link" />
+    <origin xyz="0 0.01 0.40" rpy="0.0 ${camera_tilt_angle_deg * M_PI / 180} ${M_PI/2}"/>
+  </joint>
+  <link name="camera_head_link">
     <visual>
-      <material>
-        <ambient>0.7 0.7 0.7 1</ambient>
-        <diffuse>0.7 0.7 0.7 1</diffuse>
-        <specular>0.1 0.1 0.1 1</specular>
+      <origin xyz="0 0 0" rpy="${M_PI/2} 0.0 ${M_PI/2}"/>
+      <geometry>
+        <mesh filename="file://$(find hello_mtc_with_perception)/urdf/meshes/d435.stl" />
+      </geometry>
+      <material name="aluminum">
+        <color rgba="0.5 0.5 0.5 1"/>
       </material>
     </visual>
-  </gazebo>
+    <collision>
+      <origin xyz="0 0 0" rpy="0 0 0"/>
+      <geometry>
+        <box size="${d435_cam_depth} ${d435_cam_width} ${d435_cam_height}"/>
+      </geometry>
+    </collision>
+    <inertial>
+      <mass value="0.072" />
+      <origin xyz="0 0 0" />
+      <inertia ixx="0.003881243" ixy="0.0" ixz="0.0" iyy="0.000498940" iyz="0.0" izz="0.003879257" />
+    </inertial>
+  </link>
+  <joint name="camera_head_depth_joint" type="fixed">
+    <origin xyz="0 0 0" rpy="0 0 0"/>
+    <parent link="camera_head_link"/>
+    <child link="camera_head_depth_frame" />
+  </joint>
+  <link name="camera_head_depth_frame"/>
+  <joint name="camera_head_depth_optical_joint" type="fixed">
+    <origin xyz="0 0 0" rpy="${-M_PI/2} 0 ${-M_PI/2}" />
+    <parent link="camera_head_depth_frame" />
+    <child link="camera_head_depth_optical_frame" />
+  </joint>
+  <link name="camera_head_depth_optical_frame"/>
+  <joint name="camera_head_infra1_joint" type="fixed">
+    <origin xyz="0 ${d435_cam_depth_to_infra1_offset} 0" rpy="0 0 0" />
+    <parent link="camera_head_link" />
+    <child link="camera_head_infra1_frame" />
+  </joint>
+  <link name="camera_head_infra1_frame"/>
+  <joint name="camera_head_infra1_optical_joint" type="fixed">
+    <origin xyz="0 0 0" rpy="${-M_PI/2} 0 ${-M_PI/2}" />
+    <parent link="camera_head_infra1_frame" />
+    <child link="camera_head_infra1_optical_frame" />
+  </joint>
+  <link name="camera_head_infra1_optical_frame"/>
+  <joint name="camera_head_infra2_joint" type="fixed">
+    <origin xyz="0 ${d435_cam_depth_to_infra2_offset} 0" rpy="0 0 0" />
+    <parent link="camera_head_link" />
+    <child link="camera_head_infra2_frame" />
+  </joint>
+  <link name="camera_head_infra2_frame"/>
+  <joint name="camera_head_infra2_optical_joint" type="fixed">
+    <origin xyz="0 0 0" rpy="${-M_PI/2} 0 ${-M_PI/2}" />
+    <parent link="camera_head_infra2_frame" />
+    <child link="camera_head_infra2_optical_frame" />
+  </joint>
+  <link name="camera_head_infra2_optical_frame"/>
+  <joint name="camera_head_color_joint" type="fixed">
+    <origin xyz="0 ${d435_cam_depth_to_color_offset} 0" rpy="0 0 0" />
+    <parent link="camera_head_link" />
+    <child link="camera_head_color_frame" />
+  </joint>
+  <link name="camera_head_color_frame"/>
+  <joint name="camera_head_color_optical_joint" type="fixed">
+    <origin xyz="0 0 0" rpy="${-M_PI/2} 0 ${-M_PI/2}" />
+    <parent link="camera_head_color_frame" />
+    <child link="camera_head_color_optical_frame" />
+  </joint>
+  <link name="camera_head_color_optical_frame"/>
   <gazebo reference="camera_head_link">
     <sensor name="camera_head" type="rgbd_camera">

Commit message: Got a good camera view for seeing the cylinder in the field of view for the RGBD camera

File: hello_mtc_with_perception/urdf/mycobot_280.urdf.xacro (robot description, xacro)
@@ -9,18 +9,18 @@
   <xacro:property name="d435_cam_depth_to_infra2_offset" value="-0.050"/>
   <xacro:property name="d435_cam_depth_to_color_offset" value="0.015"/>
-  <xacro:property name="camera_tilt_angle_deg" value="15"/>
+  <xacro:property name="camera_tilt_angle_deg" value="45"/>
   <link name="torso_link">
     <inertial>
-      <origin xyz="0 0 0.20" />
+      <origin xyz="0 0 0.50" />
       <mass value="2.5" />
       <inertia ixx="0.8" ixy="0.0" ixz="0.0" iyy="0.8" iyz="0.0" izz="0.8" />
     </inertial>
     <visual name="holder">
-      <origin xyz="0 0 0.20" rpy="0 0 0" />
+      <origin xyz="0 0 0.25" rpy="0 0 0" />
       <material name="LightGrey">
         <color rgba="0.7 0.7 0.7 1.0"/>
       </material>
       <geometry>
-        <cylinder radius="0.005" length="0.4"/>
+        <cylinder radius="0.005" length="0.5"/>
       </geometry>
     </visual>
@@ -35,7 +35,7 @@
     </visual>
     <collision name="holder">
-      <origin xyz="0 0 0.20" rpy="0 0 0" />
+      <origin xyz="0 0 0.25" rpy="0 0 0" />
       <geometry>
-        <cylinder radius="0.005" length="0.4"/>
+        <cylinder radius="0.005" length="0.6"/>
       </geometry>
     </collision>
@@ -50,10 +50,10 @@
     <parent link="base_link"/>
     <child link="torso_link"/>
-    <origin xyz="0.22 -0.25 0" rpy="0 0 0"/>
+    <origin xyz="0.22 -0.30 0" rpy="0 0 0"/>
   </joint>
   <joint name="camera_head_joint" type="fixed">
     <parent link="torso_link"/>
     <child link="camera_head_link" />
-    <origin xyz="0 0.01 0.40" rpy="0.0 ${camera_tilt_angle_deg * M_PI / 180} ${M_PI/2}"/>
+    <origin xyz="0 0.01 0.50" rpy="0.0 ${camera_tilt_angle_deg * M_PI / 180} ${M_PI/2}"/>
   </joint>
   <link name="camera_head_link">
@@ -144,5 +144,5 @@
       <gz_frame_id>camera_head_link</gz_frame_id>
       <topic>camera_head</topic>
-      <update_rate>5</update_rate>
+      <update_rate>10</update_rate>
       <visualize>true</visualize>
     </sensor>

Commit message: Fixed Gazebo world

File: hello_mtc_with_perception/urdf/mycobot_280.urdf.xacro (robot description, xacro)
@@ -31,5 +31,5 @@
       </material>
       <geometry>
-        <box size="0.15 0.10 0.04" />
+        <box size="0.15 0.10 0.06" />
       </geometry>
     </visual>
@@ -43,5 +43,5 @@
       <origin xyz="0 0 0.0" rpy="0 0 0" />
       <geometry>
-        <box size="0.15 0.10 0.04" />
+        <box size="0.15 0.10 0.06" />
       </geometry>
     </collision>
