Commit message: Minor changes to URDF for mycobot

File: mycobot_gazebo/urdf/ros2_control/gazebo/mycobot_280.urdf.xacro (robot description, xacro)
@@ -429,5 +429,5 @@
 	<joint name="link1_to_link2" type="revolute">
 		<axis xyz="0 0 1"/>
-		<limit effort = "${effort}" lower = "-2.879793" upper = "2.879793" velocity = "${velocity}"/>
+		<limit effort = "${effort}" lower = "-2.879793" upper = "2.879793" velocity = "${velocity}" />
 		<parent link="link1"/>
 		<child link="link2"/>
@@ -437,5 +437,5 @@
 	<joint name="link2_to_link3" type="revolute">
 		<axis xyz="0 0 1"/>
-		<limit effort = "${effort}" lower = "-2.879793" upper = "2.879793" velocity = "${velocity}"/>
+		<limit effort = "${effort}" lower = "-2.879793" upper = "2.879793" velocity = "${velocity}" />
 		<parent link="link2"/>
 		<child link="link3"/>
@@ -445,5 +445,5 @@
 	<joint name="link3_to_link4" type="revolute">
 		<axis xyz=" 0 0 1"/>
-		<limit effort = "${effort}" lower = "-2.879793" upper = "2.879793" velocity = "${velocity}"/>
+		<limit effort = "${effort}" lower = "-2.879793" upper = "2.879793" velocity = "${velocity}" />
 		<parent link="link3"/>
 		<child link="link4"/>
@@ -453,5 +453,5 @@
 	<joint name="link4_to_link5" type="revolute">
 		<axis xyz=" 0 0 1"/>
-		<limit effort = "${effort}" lower = "-2.879793" upper = "2.879793" velocity = "${velocity}"/>
+		<limit effort = "${effort}" lower = "-2.879793" upper = "2.879793" velocity = "${velocity}" />
 		<parent link="link4"/>
 		<child link="link5"/>
@@ -461,5 +461,5 @@
 	<joint name="link5_to_link6" type="revolute">
 		<axis xyz=" 0 0 1"/>
-		<limit effort = "${effort}" lower = "-2.879793" upper = "2.879793" velocity = "${velocity}"/>
+		<limit effort = "${effort}" lower = "-2.879793" upper = "2.879793" velocity = "${velocity}" />
 		<parent link="link5"/>
 		<child link="link6"/>
@@ -469,5 +469,5 @@
 	<joint name="link6_to_link6flange" type="revolute">
 		<axis xyz=" 0 0 1"/>
-		<limit effort = "${effort}" lower = "-3.05" upper = "3.05" velocity = "${velocity}"/>
+		<limit effort = "${effort}" lower = "-3.05" upper = "3.05" velocity = "${velocity}" />
 		<parent link="link6"/>
 		<child link="link6_flange"/>
@@ -482,5 +482,5 @@
 	<joint name="gripper_controller" type="revolute">
 		<axis xyz="0 0 1"/>
-		<limit effort = "${effort}" lower = "-0.7" upper = "0.15" velocity = "${velocity}"/>
+		<limit effort = "${effort}" lower = "-0.7" upper = "0.15" velocity = "${velocity}" />
 		<parent link="gripper_base"/>
 		<child link="gripper_left3"/>
@@ -490,5 +490,5 @@
 	<joint name="gripper_base_to_gripper_left2" type="revolute">
 		<axis xyz="0 0 1"/>
-		<limit effort = "${effort}" lower = "-0.8" upper = "0.5" velocity = "${velocity}"/>
+		<limit effort = "${effort}" lower = "-0.8" upper = "0.5" velocity = "${velocity}" />
 		<parent link="gripper_base"/>
 		<child link="gripper_left2"/>
@@ -499,5 +499,5 @@
 	<joint name="gripper_left3_to_gripper_left1" type="revolute">
 		<axis xyz="0 0 1"/>
-		<limit effort = "${effort}" lower = "-0.5" upper = "0.5" velocity = "${velocity}"/>
+		<limit effort = "${effort}" lower = "-0.5" upper = "0.5" velocity = "${velocity}" />
 		<parent link="gripper_left3"/>
 		<child link="gripper_left1"/>
@@ -508,5 +508,5 @@
 	<joint name="gripper_base_to_gripper_right3" type="revolute">
 		<axis xyz="0 0 1"/>
-		<limit effort = "${effort}" lower = "-0.15" upper = "0.7" velocity = "${velocity}"/>
+		<limit effort = "${effort}" lower = "-0.15" upper = "0.7" velocity = "${velocity}" />
 		<parent link="gripper_base"/>
 		<child link="gripper_right3"/>
@@ -517,5 +517,5 @@
 	<joint name="gripper_base_to_gripper_right2" type="revolute">
 		<axis xyz="0 0 1"/>
-		<limit effort = "${effort}" lower = "-0.5" upper = "0.8" velocity = "${velocity}"/>
+		<limit effort = "${effort}" lower = "-0.5" upper = "0.8" velocity = "${velocity}" />
 		<parent link="gripper_base"/>
 		<child link="gripper_right2"/>
@@ -526,5 +526,5 @@
 	<joint name="gripper_right3_to_gripper_right1" type="revolute">
 		<axis xyz="0 0 1"/>
-		<limit effort = "${effort}" lower = "-0.5" upper = "0.5" velocity = "${velocity}"/>
+		<limit effort = "${effort}" lower = "-0.5" upper = "0.5" velocity = "${velocity}" />
 		<parent link="gripper_right3"/>
 		<child link="gripper_right1"/>

Commit message: Increased effort of joints to prevent stalling

File: mycobot_gazebo/urdf/ros2_control/gazebo/mycobot_280.urdf.xacro (robot description, xacro)
@@ -4,5 +4,5 @@
     <xacro:include filename="$(find mycobot_gazebo)/urdf/ros2_control/gazebo/mycobot_280_ros2_control.xacro"/>
 	<link name="world"/>
-	<xacro:property name="effort" value="5.0"/>
+	<xacro:property name="effort" value="56.0"/>
 	<xacro:property name="velocity" value="2.792527"/>
 	<link name="base_link">
