Commit message: Renamed Xacro files for the mycobot arm

File: mycobot_description/urdf/mech/g_shape_base_v2_0.urdf.xacro (robot description, xacro)
@@ -13,5 +13,5 @@
             <visual>
                 <geometry>
-                    <mesh filename="file://$(find mycobot_description)/meshes/mycobot_280/visual/base_link.dae"/>
+                    <mesh filename="file://$(find mycobot_description)/meshes/g_shape_base_v2_0/visual/base_link.dae"/>
                 </geometry>
                 <origin xyz="0.0 0 -0.03" rpy="0 0 ${pi/2}"/>

File: mycobot_description/urdf/robots/mycobot_280.urdf.xacro (robot description, xacro)
@@ -2,10 +2,9 @@
 <robot xmlns:xacro="http://www.ros.org/wiki/xacro" name="mycobot_280">
     <xacro:arg name="add_world" default="true"/>
-    <xacro:arg name="arm_parent" default="base_link"/>
     <xacro:arg name="base_link" default="base_link"/>
     <xacro:arg name="base_type" default="g_shape"/>
-    <xacro:arg name="gripper_parent" default="base_link"/>
+    <xacro:arg name="flange_link" default="link6_flange"/>
     <xacro:arg name="gripper_type" default="adaptive_gripper"/>
-    <xacro:arg name="prefix" default=""/>
+    <xacro:arg name="prefix" default="left_"/>
     <xacro:arg name="use_gripper" default="true"/>
     <xacro:if value="$(arg add_world)">
@@ -14,20 +13,27 @@
           <parent link="world"/>
           <child link="$(arg prefix)$(arg base_link)"/>
-          <origin xyz="0 0 0.0" rpy="0 0 0"/>
+          <origin xyz="0 0 0" rpy="0 0 0"/>
       </joint>
     </xacro:if>
     <xacro:property name="current_base" value="$(arg base_type)"/>
     <xacro:if value="${current_base == 'g_shape'}">
-        <xacro:include filename="$(find mycobot_description)/urdf/mech/g_shape_base_v2_0.xacro"/>
+        <xacro:include filename="$(find mycobot_description)/urdf/mech/g_shape_base_v2_0.urdf.xacro"/>
         <xacro:g_shape_base
             base_link="$(arg base_link)"
             prefix="$(arg prefix)"/>
     </xacro:if>
+    <xacro:include filename="$(find mycobot_description)/urdf/mech/mycobot_280_arm.urdf.xacro"/>
+    <xacro:mycobot_280_arm
+      base_link="$(arg base_link)"
+      flange_link="$(arg flange_link)"
+      prefix="$(arg prefix)">
+      <origin xyz="0 0 0" rpy="0 0 0"/>
+    </xacro:mycobot_280_arm>
     <xacro:if value="$(arg use_gripper)">
         <xacro:property name="current_gripper" value="$(arg gripper_type)"/>
         <xacro:if value="${current_gripper == 'adaptive_gripper'}">
-            <xacro:include filename="$(find mycobot_description)/urdf/mech/adaptive_gripper.xacro"/>
+            <xacro:include filename="$(find mycobot_description)/urdf/mech/adaptive_gripper.urdf.xacro"/>
             <xacro:adaptive_gripper
-                parent="$(arg gripper_parent)"
+                parent="$(arg flange_link)"
                 prefix="$(arg prefix)">
                 <origin xyz="0 0 0.034" rpy="1.579 0 0"/>
