Commit message: Adjusted depth cloud angle

File: mycobot_description/urdf/sensors/intel_rgbd_cam_d435.urdf.xacro (robot description, xacro)
@@ -12,5 +12,5 @@
     <xacro:property name="d435_cam_depth_to_infra2_offset" value="-0.050"/>
     <xacro:property name="d435_cam_depth_to_color_offset" value="0.015"/>
-    <xacro:property name="camera_tilt_angle_deg" value="35"/>
+    <xacro:property name="camera_tilt_angle_deg" value="45"/>
     <link name="torso_link">
       <inertial>

Commit message: Perfect pick and place demo

File: mycobot_description/urdf/sensors/intel_rgbd_cam_d435.urdf.xacro (robot description, xacro)
@@ -12,5 +12,5 @@
     <xacro:property name="d435_cam_depth_to_infra2_offset" value="-0.050"/>
     <xacro:property name="d435_cam_depth_to_color_offset" value="0.015"/>
-    <xacro:property name="camera_tilt_angle_deg" value="45"/>
+    <xacro:property name="camera_tilt_angle_deg" value="25"/>
     <link name="torso_link">
       <inertial>
